Commit message: updates

File: model/scene_acro.xml.xacro (robot description, xacro)
@@ -56,4 +56,9 @@
       <site name="payload_connection_site" pos="0.0 0.0 0.0"/>
     </body>
+    <body name="payload_2" pos="-0.7 0.7 0.02">
+      <joint type="free" damping="0.01"/>
+      <geom type="sphere" size="0.03" rgba="0 0 1 0.8" mass="0.2"/>
+      <site name="payload_connection_site_2" pos="0.0 0.0 0.0"/>
+    </body>
     <geom name="wall_back" type="box" pos="-3 0 1.5" size="0.05 2 1.5" rgba="0.8 0.8 0.8 0.2"/>
     <geom name="wall_front" type="box" pos="8 0 1.5" size="0.05 2 1.5" rgba="0.8 0.8 0.8 0.2"/>
