Commit message: Add optional environment contacts and remove extra payload bodies

File: model/scene_acro.xml.xacro (robot description, xacro)
@@ -13,4 +13,5 @@
   <xacro:arg name="primitive_alpha" default="0.9"/>
   <xacro:arg name="simulation_timestep" default="0.0025"/>
+  <xacro:arg name="enable_environment_contacts" default="true"/>
   <xacro:arg name="imu_hz" default="350"/>
   <xacro:arg name="odom_hz" default="240"/>
@@ -30,4 +31,12 @@
   <compiler angle="radian" meshdir="$(arg meshdir)"/>
   <option timestep="$(arg simulation_timestep)" gravity="0 0 -9.81" density="1.225" viscosity="1.8e-05" integrator="RK4" />
+  <!-- Only static environment geometry uses this class; cable limits stay active. -->
+  <default>
+    <default class="environment">
+      <xacro:unless value="$(arg enable_environment_contacts)">
+        <geom contype="0" conaffinity="0"/>
+      </xacro:unless>
+    </default>
+  </default>
   <extension>
     <plugin plugin="MujocoRosUtils::WrenchToActuators"/>
@@ -57,8 +66,8 @@
     </plugin>
     <light pos="1 0 3.5" dir="0 0 -1" directional="true"/>
-    <geom name="floor" size="0 0 0.05" type="plane" material="groundplane"/>
-    <geom name="box_red" type="box" pos="2 1 0.1" size="0.2 0.2 0.1" material="mat_red" />
-    <geom name="box_green" type="box" pos="4 -1 0.1" size="0.2 0.2 0.1" material="mat_green" />
-    <geom name="box_blue" type="box" pos="6 1 0.1" size="0.2 0.2 0.1" material="mat_blue" />
+    <geom class="environment" name="floor" size="0 0 0.05" type="plane" material="groundplane"/>
+    <geom class="environment" name="box_red" type="box" pos="2 1 0.1" size="0.2 0.2 0.1" material="mat_red" />
+    <geom class="environment" name="box_green" type="box" pos="4 -1 0.1" size="0.2 0.2 0.1" material="mat_green" />
+    <geom class="environment" name="box_blue" type="box" pos="6 1 0.1" size="0.2 0.2 0.1" material="mat_blue" />
     <xacro:quadrotor_body prefix="$(arg quad_name)"
                           pos="$(arg init_x) $(arg init_y) $(arg init_z)"
@@ -81,8 +90,8 @@
       <site name="payload_connection_site_2" pos="0.0 0.0 0.0"/>
     </body>
-    <geom name="wall_back" type="box" pos="-3 0 1.5" size="0.05 2 1.5" rgba="0.8 0.8 0.8 0.2"/>
-    <geom name="wall_front" type="box" pos="8 0 1.5" size="0.05 2 1.5" rgba="0.8 0.8 0.8 0.2"/>
-    <geom name="wall_left" type="box" pos="2.5 2 1.5" size="5.5 0.05 1.5" rgba="0.8 0.8 0.8 0.2"/>
-    <geom name="wall_right" type="box" pos="2.5 -2 1.5" size="5.5 0.05 1.5" rgba="0.8 0.8 0.8 0.2"/>
+    <geom class="environment" name="wall_back" type="box" pos="-3 0 1.5" size="0.05 2 1.5" rgba="0.8 0.8 0.8 0.2"/>
+    <geom class="environment" name="wall_front" type="box" pos="8 0 1.5" size="0.05 2 1.5" rgba="0.8 0.8 0.8 0.2"/>
+    <geom class="environment" name="wall_left" type="box" pos="2.5 2 1.5" size="5.5 0.05 1.5" rgba="0.8 0.8 0.8 0.2"/>
+    <geom class="environment" name="wall_right" type="box" pos="2.5 -2 1.5" size="5.5 0.05 1.5" rgba="0.8 0.8 0.8 0.2"/>
     <geom name="origin_x" type="cylinder" fromto="0 0 0.01 0.5 0 0.01" size="0.01" rgba="1 0 0 0.1" contype="0" conaffinity="0" group="1"/>
     <geom name="origin_y" type="cylinder" fromto="0 0 0.01 0 0.5 0.01" size="0.01" rgba="0 1 0 0.1" contype="0" conaffinity="0" group="1"/>

File: model/scene_acro_gate.xml.xacro (robot description, xacro)
@@ -13,4 +13,5 @@
   <xacro:arg name="primitive_alpha" default="0.9"/>
   <xacro:arg name="simulation_timestep" default="0.0025"/>
+  <xacro:arg name="enable_environment_contacts" default="true"/>
   <xacro:arg name="imu_hz" default="350"/>
   <xacro:arg name="odom_hz" default="240"/>
@@ -30,7 +31,18 @@
   <xacro:arg name="gate_thickness" default="0.025"/>
   <xacro:property name="GATES_C" value="$(arg gates_collide)"/>
+  <xacro:unless value="$(arg enable_environment_contacts)">
+    <xacro:property name="GATES_C" value="0"/>
+  </xacro:unless>
   <xacro:include filename="quadrotor_acro_macro.xml.xacro" />
   <compiler angle="radian" meshdir="$(arg meshdir)"/>
   <option timestep="$(arg simulation_timestep)" gravity="0 0 -9.81" density="1.225" viscosity="1.8e-05" integrator="RK4" />
+  <!-- Only static environment geometry uses this class; cable limits stay active. -->
+  <default>
+    <default class="environment">
+      <xacro:unless value="$(arg enable_environment_contacts)">
+        <geom contype="0" conaffinity="0"/>
+      </xacro:unless>
+    </default>
+  </default>
   <extension>
     <plugin plugin="MujocoRosUtils::WrenchToActuators"/>
@@ -81,8 +93,8 @@
     </plugin>
     <light pos="1 0 3.5" dir="0 0 -1" directional="true"/>
-    <geom name="floor" size="0 0 0.05" type="plane" material="groundplane"/>
-    <geom name="box_red" type="box" pos="2 1 0.1" size="0.2 0.2 0.1" material="mat_red" />
-    <geom name="box_green" type="box" pos="4 -1 0.1" size="0.2 0.2 0.1" material="mat_green" />
-    <geom name="box_blue" type="box" pos="6 1 0.1" size="0.2 0.2 0.1" material="mat_blue" />
+    <geom class="environment" name="floor" size="0 0 0.05" type="plane" material="groundplane"/>
+    <geom class="environment" name="box_red" type="box" pos="2 1 0.1" size="0.2 0.2 0.1" material="mat_red" />
+    <geom class="environment" name="box_green" type="box" pos="4 -1 0.1" size="0.2 0.2 0.1" material="mat_green" />
+    <geom class="environment" name="box_blue" type="box" pos="6 1 0.1" size="0.2 0.2 0.1" material="mat_blue" />
     <xacro:quadrotor_body prefix="$(arg quad_name)"
                           pos="$(arg init_x) $(arg init_y) $(arg init_z)"
@@ -98,19 +110,12 @@
       <site name="payload_connection_site" pos="0.0 0.0 0.0"/>
     </body>
-    <body name="payload_2" pos="-0.7 0.7 0.02">
-      <joint name="payload_2_x" type="slide" axis="1 0 0" damping="0.2"/>
-      <joint name="payload_2_y" type="slide" axis="0 1 0" damping="0.2"/>
-      <joint name="payload_2_z" type="slide" axis="0 0 1" damping="0.2"/>
-      <geom type="sphere" size="0.035" rgba="0 0 1 0.8" mass="0.2"/>
-      <site name="payload_connection_site_2" pos="0.0 0.0 0.0"/>
-    </body>
     <xacro:race_gate name="gate0" px="1.5" py="0.0" pz="1.2"
                      qw="1" qx="0" qy="0" qz="0"
                      radius="$(arg gate_radius)" thickness="$(arg gate_thickness)"
                      material="mat_gate"/>
-    <geom name="wall_back" type="box" pos="-3 0 1.5" size="0.05 2 1.5" rgba="0.8 0.8 0.8 0.2"/>
-    <geom name="wall_front" type="box" pos="8 0 1.5" size="0.05 2 1.5" rgba="0.8 0.8 0.8 0.2"/>
-    <geom name="wall_left" type="box" pos="2.5 2 1.5" size="5.5 0.05 1.5" rgba="0.8 0.8 0.8 0.2"/>
-    <geom name="wall_right" type="box" pos="2.5 -2 1.5" size="5.5 0.05 1.5" rgba="0.8 0.8 0.8 0.2"/>
+    <geom class="environment" name="wall_back" type="box" pos="-3 0 1.5" size="0.05 2 1.5" rgba="0.8 0.8 0.8 0.2"/>
+    <geom class="environment" name="wall_front" type="box" pos="8 0 1.5" size="0.05 2 1.5" rgba="0.8 0.8 0.8 0.2"/>
+    <geom class="environment" name="wall_left" type="box" pos="2.5 2 1.5" size="5.5 0.05 1.5" rgba="0.8 0.8 0.8 0.2"/>
+    <geom class="environment" name="wall_right" type="box" pos="2.5 -2 1.5" size="5.5 0.05 1.5" rgba="0.8 0.8 0.8 0.2"/>
     <geom name="origin_x" type="cylinder" fromto="0 0 0.01 0.5 0 0.01" size="0.01" rgba="1 0 0 0.1" contype="0" conaffinity="0" group="1"/>
     <geom name="origin_y" type="cylinder" fromto="0 0 0.01 0 0.5 0.01" size="0.01" rgba="0 1 0 0.1" contype="0" conaffinity="0" group="1"/>

File: model/scene_acro_lidar.xml.xacro (robot description, xacro)
@@ -13,4 +13,5 @@
   <xacro:arg name="primitive_alpha" default="0.9"/>
   <xacro:arg name="simulation_timestep" default="0.0025"/>
+  <xacro:arg name="enable_environment_contacts" default="true"/>
   <xacro:arg name="imu_hz" default="350"/>
   <xacro:arg name="odom_hz" default="240"/>
@@ -29,4 +30,12 @@
   <compiler angle="radian" meshdir="$(arg meshdir)"/>
   <option timestep="$(arg simulation_timestep)" gravity="0 0 -9.81" density="1.225" viscosity="1.8e-05" integrator="RK4" />
+  <!-- Only static environment geometry uses this class; cable limits stay active. -->
+  <default>
+    <default class="environment">
+      <xacro:unless value="$(arg enable_environment_contacts)">
+        <geom contype="0" conaffinity="0"/>
+      </xacro:unless>
+    </default>
+  </default>
   <extension>
     <plugin plugin="MujocoRosUtils::WrenchToActuators"/>
@@ -60,15 +69,15 @@
     </plugin>
     <light pos="1 0 3.5" dir="0 0 -1" directional="true"/>
-    <geom name="floor" size="0 0 0.05" type="plane" material="groundplane"/>
-    <geom name="ceiling" type="box" pos="2.5 0 3.0" size="5.55 2.05 0.04" rgba="0.7 0.7 0.75 0.35"/>
-    <geom name="box_red" type="box" pos="2 1 0.1" size="0.2 0.2 0.1" material="mat_red" />
-    <geom name="box_green" type="box" pos="4 -1 0.5" size="0.2 0.2 0.5" material="mat_green" />
-    <geom name="box_blue" type="box" pos="6 1 0.5" size="0.2 0.2 0.5" material="mat_blue" />
-    <geom name="pillar_cyan" type="cylinder" pos="1.2 -1.25 0.75" size="0.12 0.75" material="mat_cyan" />
-    <geom name="pillar_yellow" type="cylinder" pos="5.2 1.35 1.1" size="0.10 1.1" material="mat_yellow" />
-    <geom name="tall_slab_left" type="box" pos="0.6 1.35 0.8" size="0.08 0.35 0.8" material="mat_gray" />
-    <geom name="low_crate_back" type="box" pos="6.7 -0.8 0.25" size="0.28 0.32 0.25" material="mat_cyan" />
-    <geom name="overhead_beam" type="box" pos="3.6 1.1 1.8" size="0.9 0.08 0.08" material="mat_gray" />
-    <geom name="offset_panel" type="box" pos="7.1 0.25 1.05" size="0.08 0.55 1.05" material="mat_red" />
+    <geom class="environment" name="floor" size="0 0 0.05" type="plane" material="groundplane"/>
+    <geom class="environment" name="ceiling" type="box" pos="2.5 0 3.0" size="5.55 2.05 0.04" rgba="0.7 0.7 0.75 0.35"/>
+    <geom class="environment" name="box_red" type="box" pos="2 1 0.1" size="0.2 0.2 0.1" material="mat_red" />
+    <geom class="environment" name="box_green" type="box" pos="4 -1 0.5" size="0.2 0.2 0.5" material="mat_green" />
+    <geom class="environment" name="box_blue" type="box" pos="6 1 0.5" size="0.2 0.2 0.5" material="mat_blue" />
+    <geom class="environment" name="pillar_cyan" type="cylinder" pos="1.2 -1.25 0.75" size="0.12 0.75" material="mat_cyan" />
+    <geom class="environment" name="pillar_yellow" type="cylinder" pos="5.2 1.35 1.1" size="0.10 1.1" material="mat_yellow" />
+    <geom class="environment" name="tall_slab_left" type="box" pos="0.6 1.35 0.8" size="0.08 0.35 0.8" material="mat_gray" />
+    <geom class="environment" name="low_crate_back" type="box" pos="6.7 -0.8 0.25" size="0.28 0.32 0.25" material="mat_cyan" />
+    <geom class="environment" name="overhead_beam" type="box" pos="3.6 1.1 1.8" size="0.9 0.08 0.08" material="mat_gray" />
+    <geom class="environment" name="offset_panel" type="box" pos="7.1 0.25 1.05" size="0.08 0.55 1.05" material="mat_red" />
     <xacro:quadrotor_body prefix="$(arg quad_name)"
                           pos="$(arg init_x) $(arg init_y) $(arg init_z)"
@@ -92,8 +101,8 @@
       <site name="payload_connection_site_2" pos="0.0 0.0 0.0"/>
     </body>
-    <geom name="wall_back" type="box" pos="-3 0 1.5" size="0.05 2 1.5" rgba="0.8 0.8 0.8 0.2"/>
-    <geom name="wall_front" type="box" pos="8 0 1.5" size="0.05 2 1.5" rgba="0.8 0.8 0.8 0.2"/>
-    <geom name="wall_left" type="box" pos="2.5 2 1.5" size="5.5 0.05 1.5" rgba="0.8 0.8 0.8 0.2"/>
-    <geom name="wall_right" type="box" pos="2.5 -2 1.5" size="5.5 0.05 1.5" rgba="0.8 0.8 0.8 0.2"/>
+    <geom class="environment" name="wall_back" type="box" pos="-3 0 1.5" size="0.05 2 1.5" rgba="0.8 0.8 0.8 0.2"/>
+    <geom class="environment" name="wall_front" type="box" pos="8 0 1.5" size="0.05 2 1.5" rgba="0.8 0.8 0.8 0.2"/>
+    <geom class="environment" name="wall_left" type="box" pos="2.5 2 1.5" size="5.5 0.05 1.5" rgba="0.8 0.8 0.8 0.2"/>
+    <geom class="environment" name="wall_right" type="box" pos="2.5 -2 1.5" size="5.5 0.05 1.5" rgba="0.8 0.8 0.8 0.2"/>
     <geom name="origin_x" type="cylinder" fromto="0 0 0.01 0.5 0 0.01" size="0.01" rgba="1 0 0 0.1" contype="0" conaffinity="0" group="1"/>
     <geom name="origin_y" type="cylinder" fromto="0 0 0.01 0 0.5 0.01" size="0.01" rgba="0 1 0 0.1" contype="0" conaffinity="0" group="1"/>

File: model/scene_acro_payload.xml.xacro (robot description, xacro)
@@ -22,4 +22,5 @@
   <xacro:arg name="primitive_alpha" default="0.9"/>
   <xacro:arg name="simulation_timestep" default="0.0025"/>
+  <xacro:arg name="enable_environment_contacts" default="true"/>
   <xacro:arg name="imu_hz" default="350"/>
   <xacro:arg name="odom_hz" default="240"/>
@@ -38,4 +39,12 @@
   <compiler angle="radian" meshdir="$(arg meshdir)"/>
   <option timestep="$(arg simulation_timestep)" gravity="0 0 -9.81" density="1.225" viscosity="1.8e-05" integrator="RK4" />
+  <!-- Only static environment geometry uses this class; cable limits stay active. -->
+  <default>
+    <default class="environment">
+      <xacro:unless value="$(arg enable_environment_contacts)">
+        <geom contype="0" conaffinity="0"/>
+      </xacro:unless>
+    </default>
+  </default>
   <extension>
     <plugin plugin="MujocoRosUtils::WrenchToActuators"/>
@@ -65,8 +74,8 @@
     </plugin>
     <light pos="1 0 3.5" dir="0 0 -1" directional="true"/>
-    <geom name="floor" size="0 0 0.05" type="plane" material="groundplane"/>
-    <geom name="box_red" type="box" pos="2 1 0.1" size="0.2 0.2 0.1" material="mat_red" />
-    <geom name="box_green" type="box" pos="4 -1 0.1" size="0.2 0.2 0.1" material="mat_green" />
-    <geom name="box_blue" type="box" pos="6 1 0.1" size="0.2 0.2 0.1" material="mat_blue" />
+    <geom class="environment" name="floor" size="0 0 0.05" type="plane" material="groundplane"/>
+    <geom class="environment" name="box_red" type="box" pos="2 1 0.1" size="0.2 0.2 0.1" material="mat_red" />
+    <geom class="environment" name="box_green" type="box" pos="4 -1 0.1" size="0.2 0.2 0.1" material="mat_green" />
+    <geom class="environment" name="box_blue" type="box" pos="6 1 0.1" size="0.2 0.2 0.1" material="mat_blue" />
     <xacro:quadrotor_body prefix="$(arg quad_name)"
                           pos="$(arg init_x) $(arg init_y) $(arg init_z)"
@@ -86,15 +95,8 @@
       <site name="payload_connection_site" pos="0.0 0.0 0.0"/>
     </body>
-    <body name="payload_2" pos="-0.7 0.7 0.02">
-      <joint name="payload_2_x" type="slide" axis="1 0 0" damping="0.06"/>
-      <joint name="payload_2_y" type="slide" axis="0 1 0" damping="0.06"/>
-      <joint name="payload_2_z" type="slide" axis="0 0 1" damping="0.06"/>
-      <geom type="sphere" size="0.035" rgba="0 0 1 0.8" mass="0.2"/>
-      <site name="payload_connection_site_2" pos="0.0 0.0 0.0"/>
-    </body>
-    <geom name="wall_back" type="box" pos="-3 0 1.5" size="0.05 2 1.5" rgba="0.8 0.8 0.8 0.2"/>
-    <geom name="wall_front" type="box" pos="8 0 1.5" size="0.05 2 1.5" rgba="0.8 0.8 0.8 0.2"/>
-    <geom name="wall_left" type="box" pos="2.5 2 1.5" size="5.5 0.05 1.5" rgba="0.8 0.8 0.8 0.2"/>
-    <geom name="wall_right" type="box" pos="2.5 -2 1.5" size="5.5 0.05 1.5" rgba="0.8 0.8 0.8 0.2"/>
+    <geom class="environment" name="wall_back" type="box" pos="-3 0 1.5" size="0.05 2 1.5" rgba="0.8 0.8 0.8 0.2"/>
+    <geom class="environment" name="wall_front" type="box" pos="8 0 1.5" size="0.05 2 1.5" rgba="0.8 0.8 0.8 0.2"/>
+    <geom class="environment" name="wall_left" type="box" pos="2.5 2 1.5" size="5.5 0.05 1.5" rgba="0.8 0.8 0.8 0.2"/>
+    <geom class="environment" name="wall_right" type="box" pos="2.5 -2 1.5" size="5.5 0.05 1.5" rgba="0.8 0.8 0.8 0.2"/>
     <geom name="origin_x" type="cylinder" fromto="0 0 0.01 0.5 0 0.01" size="0.01" rgba="1 0 0 0.1" contype="0" conaffinity="0" group="1"/>
     <geom name="origin_y" type="cylinder" fromto="0 0 0.01 0 0.5 0.01" size="0.01" rgba="0 1 0 0.1" contype="0" conaffinity="0" group="1"/>

File: model/scene_acro_payload_lidar.xml.xacro (robot description, xacro)
@@ -13,4 +13,5 @@
   <xacro:arg name="primitive_alpha" default="0.9"/>
   <xacro:arg name="simulation_timestep" default="0.0025"/>
+  <xacro:arg name="enable_environment_contacts" default="true"/>
   <xacro:arg name="imu_hz" default="350"/>
   <xacro:arg name="odom_hz" default="240"/>
@@ -29,4 +30,12 @@
   <compiler angle="radian" meshdir="$(arg meshdir)"/>
   <option timestep="$(arg simulation_timestep)" gravity="0 0 -9.81" density="1.225" viscosity="1.8e-05" integrator="RK4" />
+  <!-- Only static environment geometry uses this class; cable limits stay active. -->
+  <default>
+    <default class="environment">
+      <xacro:unless value="$(arg enable_environment_contacts)">
+        <geom contype="0" conaffinity="0"/>
+      </xacro:unless>
+    </default>
+  </default>
   <extension>
     <plugin plugin="MujocoRosUtils::WrenchToActuators"/>
@@ -60,14 +69,14 @@
     </plugin>
     <light pos="1 0 3.5" dir="0 0 -1" directional="true"/>
-    <geom name="floor" size="0 0 0.05" type="plane" material="groundplane"/>
-    <geom name="ceiling" type="box" pos="2.5 0 3.0" size="5.55 2.05 0.04" rgba="0.7 0.7 0.75 0.35"/>
-    <geom name="box_red" type="box" pos="2 1 0.1" size="0.2 0.2 0.1" material="mat_red" />
-    <geom name="box_blue" type="box" pos="6 1 0.5" size="0.2 0.2 0.5" material="mat_blue" />
-    <geom name="pillar_cyan" type="cylinder" pos="1.2 -1.25 0.75" size="0.12 0.75" material="mat_cyan" />
-    <geom name="pillar_yellow" type="cylinder" pos="5.2 1.35 1.1" size="0.10 1.1" material="mat_yellow" />
-    <geom name="tall_slab_left" type="box" pos="0.6 1.35 0.8" size="0.08 0.35 0.8" material="mat_gray" />
-    <geom name="low_crate_back" type="box" pos="6.7 -0.8 0.25" size="0.28 0.32 0.25" material="mat_cyan" />
-    <geom name="overhead_beam" type="box" pos="3.6 1.1 1.8" size="0.9 0.08 0.08" material="mat_gray" />
-    <geom name="offset_panel" type="box" pos="7.1 0.25 1.05" size="0.08 0.55 1.05" material="mat_red" />
+    <geom class="environment" name="floor" size="0 0 0.05" type="plane" material="groundplane"/>
+    <geom class="environment" name="ceiling" type="box" pos="2.5 0 3.0" size="5.55 2.05 0.04" rgba="0.7 0.7 0.75 0.35"/>
+    <geom class="environment" name="box_red" type="box" pos="2 1 0.1" size="0.2 0.2 0.1" material="mat_red" />
+    <geom class="environment" name="box_blue" type="box" pos="6 1 0.5" size="0.2 0.2 0.5" material="mat_blue" />
+    <geom class="environment" name="pillar_cyan" type="cylinder" pos="1.2 -1.25 0.75" size="0.12 0.75" material="mat_cyan" />
+    <geom class="environment" name="pillar_yellow" type="cylinder" pos="5.2 1.35 1.1" size="0.10 1.1" material="mat_yellow" />
+    <geom class="environment" name="tall_slab_left" type="box" pos="0.6 1.35 0.8" size="0.08 0.35 0.8" material="mat_gray" />
+    <geom class="environment" name="low_crate_back" type="box" pos="6.7 -0.8 0.25" size="0.28 0.32 0.25" material="mat_cyan" />
+    <geom class="environment" name="overhead_beam" type="box" pos="3.6 1.1 1.8" size="0.9 0.08 0.08" material="mat_gray" />
+    <geom class="environment" name="offset_panel" type="box" pos="7.1 0.25 1.05" size="0.08 0.55 1.05" material="mat_red" />
     <xacro:quadrotor_body prefix="$(arg quad_name)"
                           pos="$(arg init_x) $(arg init_y) $(arg init_z)"
@@ -84,15 +93,8 @@
       <site name="payload_connection_site" pos="0.0 0.0 0.0"/>
     </body>
-    <body name="payload_2" pos="-0.7 0.7 0.02">
-      <joint name="payload_2_x" type="slide" axis="1 0 0" damping="0.06"/>
-      <joint name="payload_2_y" type="slide" axis="0 1 0" damping="0.06"/>
-      <joint name="payload_2_z" type="slide" axis="0 0 1" damping="0.06"/>
-      <geom type="sphere" size="0.035" rgba="0 0 1 0.8" mass="0.2"/>
-      <site name="payload_connection_site_2" pos="0.0 0.0 0.0"/>
-    </body>
-    <geom name="wall_back" type="box" pos="-3 0 1.5" size="0.05 2 1.5" rgba="0.8 0.8 0.8 0.2"/>
-    <geom name="wall_front" type="box" pos="8 0 1.5" size="0.05 2 1.5" rgba="0.8 0.8 0.8 0.2"/>
-    <geom name="wall_left" type="box" pos="2.5 2 1.5" size="5.5 0.05 1.5" rgba="0.8 0.8 0.8 0.2"/>
-    <geom name="wall_right" type="box" pos="2.5 -2 1.5" size="5.5 0.05 1.5" rgba="0.8 0.8 0.8 0.2"/>
+    <geom class="environment" name="wall_back" type="box" pos="-3 0 1.5" size="0.05 2 1.5" rgba="0.8 0.8 0.8 0.2"/>
+    <geom class="environment" name="wall_front" type="box" pos="8 0 1.5" size="0.05 2 1.5" rgba="0.8 0.8 0.8 0.2"/>
+    <geom class="environment" name="wall_left" type="box" pos="2.5 2 1.5" size="5.5 0.05 1.5" rgba="0.8 0.8 0.8 0.2"/>
+    <geom class="environment" name="wall_right" type="box" pos="2.5 -2 1.5" size="5.5 0.05 1.5" rgba="0.8 0.8 0.8 0.2"/>
     <geom name="origin_x" type="cylinder" fromto="0 0 0.01 0.5 0 0.01" size="0.01" rgba="1 0 0 0.1" contype="0" conaffinity="0" group="1"/>
     <geom name="origin_y" type="cylinder" fromto="0 0 0.01 0 0.5 0.01" size="0.01" rgba="0 1 0 0.1" contype="0" conaffinity="0" group="1"/>
