Commit message: updates

File: model/quadrotor_acro_macro.xml.xacro (robot description, xacro)
@@ -18,5 +18,5 @@
       <site name="${prefix}_rateY" type="box" pos="0 0 0" size="0.035 0.035 0.015" rgba="0 1 1 1"/>
       <site name="${prefix}_rateZ" type="box" pos="0 0 0" size="0.035 0.035 0.015" rgba="0 1 1 1"/>
-      <site name="${prefix}_payload_site" pos="0.0 0.0 -0.08"/>
+      <site name="${prefix}_payload_site" pos="0.0 0.0 -0.05"/>
       <camera name="${prefix}_camera" pos="0.035 0 -0.015" euler="0 0 -1.57"/>
     </body>

File: model/quadrotor_lowlevel_macro.xml.xacro (robot description, xacro)
@@ -18,5 +18,5 @@
       <site name="${prefix}_rateY" type="box" pos="0 0 0" size="0.035 0.035 0.015" rgba="0 1 1 1"/>
       <site name="${prefix}_rateZ" type="box" pos="0 0 0" size="0.035 0.035 0.015" rgba="0 1 1 1"/>
-      <site name="${prefix}_payload_site" pos="0.0 0.0 0.0"/>
+      <site name="${prefix}_payload_site" pos="0.0 0.0 -0.08"/>
       <camera name="${prefix}_camera" pos="0.035 0 -0.015" euler="0 0 -1.57"/>
     </body>

File: model/scene_acro.xml.xacro (robot description, xacro)
@@ -20,21 +20,20 @@
   </extension>
   <asset>
-    <texture name="texwood" type="2d" builtin="gradient" width="512" height="512"
-             rgb1="0.80 0.65 0.45" rgb2="0.65 0.50 0.35" />
-    <material name="matwood" texture="texwood" texrepeat="1 15"
-              reflectance="0.02" shininess="0.05" specular="0.1" />
     <material name="mat_red"   rgba="0.8 0.1 0.1 1" reflectance="0.01" shininess="0.01" specular="0.0" />
     <material name="mat_green" rgba="0.1 0.8 0.1 1" reflectance="0.01" shininess="0.01" specular="0.0" />
     <material name="mat_blue"  rgba="0.1 0.1 0.8 1" reflectance="0.01" shininess="0.01" specular="0.0" />
+    <texture type="skybox" builtin="flat" rgb1="0 0 0" rgb2="0 0 0" width="512" height="3072"/>
+    <texture type="2d" name="groundplane" builtin="checker" mark="edge" rgb1="0.2 0.3 0.4" rgb2="0.1 0.2 0.3" markrgb="0.8 0.8 0.8" width="300" height="300"/>
+    <material name="groundplane" texture="groundplane" texuniform="true" texrepeat="5 5" reflectance="0.2"/>
   </asset>
   <worldbody>
-    <light pos="0 0 1.5" dir="0 0 -1" directional="true"/>
-    <geom name="floor" type="box" pos="2.5 0 -0.05" size="5.5 2 0.05" material="matwood" condim="3"/>
+    <light pos="1 0 3.5" dir="0 0 -1" directional="true"/>
+    <geom name="floor" size="0 0 0.05" type="plane" material="groundplane"/>
     <geom name="box_red" type="box" pos="2 1 0.1" size="0.2 0.2 0.1" material="mat_red" />
     <geom name="box_green" type="box" pos="4 -1 0.1" size="0.2 0.2 0.1" material="mat_green" />
     <geom name="box_blue" type="box" pos="6 1 0.1" size="0.2 0.2 0.1" material="mat_blue" />
     <xacro:quadrotor_body prefix="$(arg quad_name)" pos="$(arg init_x) $(arg init_y) $(arg init_z)" euler="$(arg init_roll) $(arg init_pitch) $(arg init_yaw)" />
-    <body name="payload" pos="0.6 0 0.02">
-      <joint type="free" damping="0.001"/>
+    <body name="payload" pos="0.8 0 0.02">
+      <joint type="free" damping="0.01"/>
       <geom type="sphere" size="0.03" rgba="0 0 1 0.8" mass="0.1128"/>
       <site name="payload_connection_site" pos="0.0 0.0 0.03"/>
@@ -61,5 +60,5 @@
   </sensor>
   <tendon>
-    <spatial name="rope0" limited="true" range="0 0.6" width=".0005">
+    <spatial name="rope0" limited="true" range="0 0.8" width=".0005">
       <site site="$(arg quad_name)_payload_site"/>
       <site site="payload_connection_site"/>

File: model/scene_acro_humanoid.xml.xacro (robot description, xacro)
@@ -8,8 +8,7 @@
   <xacro:arg name="init_pitch" default="0.0"/>
   <xacro:arg name="init_yaw"   default="0.0"/>
-  <xacro:arg name="ctrl_mode" default="acro"/>
   <xacro:include filename="quadrotor_acro_macro.xml.xacro" />
-  <xacro:include filename="quadrotor_lowlevel_macro.xml.xacro" />
-  <compiler angle="radian"/>
+  <xacro:include filename="humanoid_macro.xml.xacro"/>
+  <compiler angle="radian" meshdir="/home/fer/payload_transportation_ws/src/acp_mujoco_simulator/model/humanoid_resource/meshes"/>
   <option timestep="0.003" gravity="0 0 -9.81" density="1.225" viscosity="1.8e-05" integrator="RK4" />
   <extension>
@@ -22,22 +21,23 @@
   </extension>
   <asset>
-    <texture name="texwood" type="2d" builtin="gradient" width="512" height="512"
-             rgb1="0.80 0.65 0.45" rgb2="0.65 0.50 0.35" />
-    <material name="matwood" texture="texwood" texrepeat="1 15"
-              reflectance="0.02" shininess="0.05" specular="0.1" />
     <material name="mat_red"   rgba="0.8 0.1 0.1 1" reflectance="0.01" shininess="0.01" specular="0.0" />
     <material name="mat_green" rgba="0.1 0.8 0.1 1" reflectance="0.01" shininess="0.01" specular="0.0" />
     <material name="mat_blue"  rgba="0.1 0.1 0.8 1" reflectance="0.01" shininess="0.01" specular="0.0" />
+    <texture type="skybox" builtin="flat" rgb1="0 0 0" rgb2="0 0 0" width="512" height="3072"/>
+    <texture type="2d" name="groundplane" builtin="checker" mark="edge" rgb1="0.2 0.3 0.4" rgb2="0.1 0.2 0.3" markrgb="0.8 0.8 0.8" width="300" height="300"/>
+    <material name="groundplane" texture="groundplane" texuniform="true" texrepeat="5 5" reflectance="0.2"/>
+    <xacro:g1_humanoid_assets prefix="g1"/>
   </asset>
   <worldbody>
-    <light pos="0 0 1.5" dir="0 0 -1" directional="true"/>
-    <geom name="floor" type="box" pos="2.5 0 -0.05" size="5.5 2 0.05" material="matwood" condim="3"/>
+    <light pos="1 0 3.5" dir="0 0 -1" directional="true"/>
+    <geom name="floor" size="0 0 0.05" type="plane" material="groundplane"/>
     <geom name="box_red" type="box" pos="2 1 0.1" size="0.2 0.2 0.1" material="mat_red" />
     <geom name="box_green" type="box" pos="4 -1 0.1" size="0.2 0.2 0.1" material="mat_green" />
     <geom name="box_blue" type="box" pos="6 1 0.1" size="0.2 0.2 0.1" material="mat_blue" />
     <xacro:quadrotor_body prefix="$(arg quad_name)" pos="$(arg init_x) $(arg init_y) $(arg init_z)" euler="$(arg init_roll) $(arg init_pitch) $(arg init_yaw)" />
-    <body name="payload" pos="1 0 0.02">
-      <joint type="free" damping="0.001"/>
-      <geom type="sphere" size="0.03" rgba="0 0 1 0.8" mass="0.1"/>
+    <xacro:g1_humanoid_body prefix="g1" pos="3 0 0.793" euler="0 0 0"/>
+    <body name="payload" pos="0.8 0 0.02">
+      <joint type="free" damping="0.01"/>
+      <geom type="sphere" size="0.03" rgba="0 0 1 0.8" mass="0.1128"/>
       <site name="payload_connection_site" pos="0.0 0.0 0.03"/>
     </body>
@@ -63,5 +63,5 @@
   </sensor>
   <tendon>
-    <spatial name="rope0" limited="true" range="0 1" width=".0005">
+    <spatial name="rope0" limited="true" range="0 0.8" width=".0005">
       <site site="$(arg quad_name)_payload_site"/>
       <site site="payload_connection_site"/>

Commit message: include mesh reduce performance mujoco

File: model/quadrotor_acro_macro.xml.xacro (robot description, xacro)
@@ -1,21 +1,27 @@
 <?xml version="1.0"?>
 <mujoco xmlns:xacro="http://www.ros.org/wiki/xacro">
-  <xacro:macro name="quadrotor_body" params="prefix pos euler:='0 0 0'">
+  <xacro:macro name="quadrotor_visual_assets">
+    <mesh name="quadrotor_visual_mesh" file="raxl_assembly.obj" scale="0.001 0.001 0.001" />
+  </xacro:macro>
+  <xacro:macro name="quadrotor_body" params="prefix pos euler:='0 0 0' mesh_pos:='-0.17 -0.16 -0.1' mesh_euler:='0 1.57 1.57079632679' primitive_alpha:='0'">
     <body name="${prefix}" pos="${pos}" euler="${euler}">
       <joint name="${prefix}" type="free" damping="0.001" armature="0" pos="0 0 0"/>
-      <geom name="${prefix}_core" type="box" size="0.035 0.035 0.015" rgba="1.0 1.0 0.0 1.0" mass=".85"/>
+      <geom name="${prefix}_visual_mesh" type="mesh" mesh="quadrotor_visual_mesh"
+            pos="${mesh_pos}" euler="${mesh_euler}"
+            rgba="0.1 0.1 0.1 1" contype="0" conaffinity="0" density="0"/>
+      <geom name="${prefix}_core" type="box" size="0.035 0.035 0.015" rgba="1.0 1.0 0.0 ${primitive_alpha}" mass=".85"/>
       <site name="${prefix}_imu" pos="0 0 0"/>
-      <geom name="${prefix}_a00" type="box" pos=".071 0.071 0.0" size="0.05 0.01 0.0025" quat=".924 0 0 0.383" rgba="1 0.5 0 1" mass=".035"/>
-      <geom name="${prefix}_a10" type="box" pos=".071 -0.071 0.0" size="0.05 0.01 0.0025" quat=".383 0 0 0.924" rgba="1 0.5 0 1" mass=".035"/>
-      <geom name="${prefix}_a20" type="box" pos="-0.071 -0.071 0.0" size="0.05 0.01 0.0025" quat="-.383 0 0 0.924" rgba="1 0.5 0 1" mass=".035"/>
-      <geom name="${prefix}_a30" type="box" pos="-.071 0.071 0.0" size="0.05 0.01 0.0025" quat=".924 0 0 -0.383" rgba="1 0.5 0 1" mass=".035"/>
-      <geom name="${prefix}_thruster00" type="cylinder" pos="0.1 0.1 0.01" size="0.03 0.0025" quat="1.0 0.0 0.0 0." rgba="0.0 0.0 0.0 1.0" mass=".015"/>
-      <geom name="${prefix}_thruster10" type="cylinder" pos="0.1 -0.1 0.01" size="0.03 0.0025" quat="1.0 0.0 0.0 0." rgba="0.0 0.0 0.0 1.0" mass=".015"/>
-      <geom name="${prefix}_thruster20" type="cylinder" pos="-0.1 -0.1 0.01" size="0.03 0.0025" quat="1.0 0.0 0.0 0." rgba="0.0 0.0 0.0 1.0" mass=".015"/>
-      <geom name="${prefix}_thruster30" type="cylinder" pos="-0.1 0.1 0.01" size="0.03 0.0025" quat="1.0 0.0 0.0 0." rgba="0.0 0.0 0.0 1.0" mass=".015"/>
-      <site name="${prefix}_thrust" type="box" pos="0 0 0" size="0.035 0.035 0.015" rgba="0 1 1 1"/>
-      <site name="${prefix}_rateX" type="box" pos="0 0 0" size="0.035 0.035 0.015" rgba="0 1 1 1"/>
-      <site name="${prefix}_rateY" type="box" pos="0 0 0" size="0.035 0.035 0.015" rgba="0 1 1 1"/>
-      <site name="${prefix}_rateZ" type="box" pos="0 0 0" size="0.035 0.035 0.015" rgba="0 1 1 1"/>
+      <geom name="${prefix}_a00" type="box" pos=".071 0.071 0.0" size="0.05 0.01 0.0025" quat=".924 0 0 0.383" rgba="1 0.5 0 ${primitive_alpha}" mass=".035"/>
+      <geom name="${prefix}_a10" type="box" pos=".071 -0.071 0.0" size="0.05 0.01 0.0025" quat=".383 0 0 0.924" rgba="1 0.5 0 ${primitive_alpha}" mass=".035"/>
+      <geom name="${prefix}_a20" type="box" pos="-0.071 -0.071 0.0" size="0.05 0.01 0.0025" quat="-.383 0 0 0.924" rgba="1 0.5 0 ${primitive_alpha}" mass=".035"/>
+      <geom name="${prefix}_a30" type="box" pos="-.071 0.071 0.0" size="0.05 0.01 0.0025" quat=".924 0 0 -0.383" rgba="1 0.5 0 ${primitive_alpha}" mass=".035"/>
+      <geom name="${prefix}_thruster00" type="cylinder" pos="0.1 0.1 0.01" size="0.03 0.0025" quat="1.0 0.0 0.0 0." rgba="0.0 0.0 0.0 ${primitive_alpha}" mass=".015"/>
+      <geom name="${prefix}_thruster10" type="cylinder" pos="0.1 -0.1 0.01" size="0.03 0.0025" quat="1.0 0.0 0.0 0." rgba="0.0 0.0 0.0 ${primitive_alpha}" mass=".015"/>
+      <geom name="${prefix}_thruster20" type="cylinder" pos="-0.1 -0.1 0.01" size="0.03 0.0025" quat="1.0 0.0 0.0 0." rgba="0.0 0.0 0.0 ${primitive_alpha}" mass=".015"/>
+      <geom name="${prefix}_thruster30" type="cylinder" pos="-0.1 0.1 0.01" size="0.03 0.0025" quat="1.0 0.0 0.0 0." rgba="0.0 0.0 0.0 ${primitive_alpha}" mass=".015"/>
+      <site name="${prefix}_thrust" type="box" pos="0 0 0" size="0.035 0.035 0.015" rgba="0 1 1 ${primitive_alpha}"/>
+      <site name="${prefix}_rateX" type="box" pos="0 0 0" size="0.035 0.035 0.015" rgba="0 1 1 ${primitive_alpha}"/>
+      <site name="${prefix}_rateY" type="box" pos="0 0 0" size="0.035 0.035 0.015" rgba="0 1 1 ${primitive_alpha}"/>
+      <site name="${prefix}_rateZ" type="box" pos="0 0 0" size="0.035 0.035 0.015" rgba="0 1 1 ${primitive_alpha}"/>
       <site name="${prefix}_payload_site" pos="0.0 0.0 -0.05"/>
     </body>

File: model/scene_acro.xml.xacro (robot description, xacro)
@@ -8,6 +8,10 @@
   <xacro:arg name="init_pitch" default="0.0"/>
   <xacro:arg name="init_yaw"   default="0.0"/>
+  <xacro:arg name="meshdir" default="."/>
+  <xacro:arg name="mesh_pos" default="-0.17 -0.16 -0.1"/>
+  <xacro:arg name="mesh_euler" default="0 1.57 1.57079632679"/>
+  <xacro:arg name="primitive_alpha" default="0.0"/>
   <xacro:include filename="quadrotor_acro_macro.xml.xacro" />
-  <compiler angle="radian"/>
+  <compiler angle="radian" meshdir="$(arg meshdir)"/>
   <option timestep="0.002" gravity="0 0 -9.81" density="1.225" viscosity="1.8e-05" integrator="RK4" />
   <extension>
@@ -25,4 +29,5 @@
     <material name="mat_green" rgba="0.1 0.8 0.1 1" reflectance="0.01" shininess="0.01" specular="0.0" />
     <material name="mat_blue"  rgba="0.1 0.1 0.8 1" reflectance="0.01" shininess="0.01" specular="0.0" />
+    <xacro:quadrotor_visual_assets />
     <texture type="skybox" builtin="flat" rgb1="0 0 0" rgb2="0 0 0" width="512" height="3072"/>
     <texture type="2d" name="groundplane" builtin="checker" mark="edge" rgb1="0.2 0.3 0.4" rgb2="0.1 0.2 0.3" markrgb="0.8 0.8 0.8" width="300" height="300"/>
@@ -40,5 +45,10 @@
     <geom name="box_green" type="box" pos="4 -1 0.1" size="0.2 0.2 0.1" material="mat_green" />
     <geom name="box_blue" type="box" pos="6 1 0.1" size="0.2 0.2 0.1" material="mat_blue" />
-    <xacro:quadrotor_body prefix="$(arg quad_name)" pos="$(arg init_x) $(arg init_y) $(arg init_z)" euler="$(arg init_roll) $(arg init_pitch) $(arg init_yaw)" />
+    <xacro:quadrotor_body prefix="$(arg quad_name)"
+                          pos="$(arg init_x) $(arg init_y) $(arg init_z)"
+                          euler="$(arg init_roll) $(arg init_pitch) $(arg init_yaw)"
+                          mesh_pos="$(arg mesh_pos)"
+                          mesh_euler="$(arg mesh_euler)"
+                          primitive_alpha="$(arg primitive_alpha)" />
     <body name="payload" pos="0.7 0.0 0.02">
       <joint type="free" damping="0.01"/>

Commit message: multiples quadrotors

File: model/quadrotor_acro_macro.xml.xacro (robot description, xacro)
@@ -7,7 +7,8 @@
     <body name="${prefix}" pos="${pos}" euler="${euler}">
       <joint name="${prefix}" type="free" damping="0.001" armature="0" pos="0 0 0"/>
-      <geom name="${prefix}_visual_mesh" type="mesh" mesh="quadrotor_visual_mesh"
+      <!-- This is only to visual purposes -->
+      <!--<geom name="${prefix}_visual_mesh" type="mesh" mesh="quadrotor_visual_mesh"
             pos="${mesh_pos}" euler="${mesh_euler}"
-            rgba="0.1 0.1 0.1 1" contype="0" conaffinity="0" density="0"/>
+            rgba="0.1 0.1 0.1 1" contype="0" conaffinity="0" density="0"/>-->
       <geom name="${prefix}_core" type="box" size="0.035 0.035 0.015" rgba="1.0 1.0 0.0 ${primitive_alpha}" mass="1.04"
             solref=".5e-4" solimp="0.9 0.99 1e-4" fluidcoef="0.5 0.25 0.5 2.0 1.0"/>

File: model/scene_acro_point_mass_multiple.xml.xacro (robot description, xacro)
@@ -1,15 +1,8 @@
 <?xml version="1.0"?>
 <mujoco xmlns:xacro="http://www.ros.org/wiki/xacro" model="Multi-Drone Scene">
-  <xacro:arg name="quad_name" default="quadrotor"/>
-  <xacro:arg name="init_x" default="0.0"/>
-  <xacro:arg name="init_y" default="0.0"/>
-  <xacro:arg name="init_z" default="0.02"/>
-  <xacro:arg name="init_roll"  default="0.0"/>
-  <xacro:arg name="init_pitch" default="0.0"/>
-  <xacro:arg name="init_yaw"   default="0.0"/>
   <xacro:arg name="meshdir" default="."/>
   <xacro:arg name="mesh_pos" default="-0.17 -0.16 -0.1"/>
   <xacro:arg name="mesh_euler" default="0 1.57 1.57079632679"/>
-  <xacro:arg name="primitive_alpha" default="0.9"/>
+  <xacro:arg name="primitive_alpha" default="0.8"/>
   <xacro:include filename="quadrotor_acro_macro.xml.xacro" />
   <compiler angle="radian" meshdir="$(arg meshdir)"/>
@@ -45,20 +38,6 @@
     <geom name="box_green" type="box" pos="4 -1 0.1" size="0.2 0.2 0.1" material="mat_green" />
     <geom name="box_blue" type="box" pos="6 1 0.1" size="0.2 0.2 0.1" material="mat_blue" />
-    <xacro:quadrotor_body prefix="$(arg quad_name)"
-                          pos="$(arg init_x) $(arg init_y) $(arg init_z)"
-                          euler="$(arg init_roll) $(arg init_pitch) $(arg init_yaw)"
-                          mesh_pos="$(arg mesh_pos)"
-                          mesh_euler="$(arg mesh_euler)"
-                          primitive_alpha="$(arg primitive_alpha)" />
-    <body name="payload" pos="-0.7 0.0 0.02">
-      <joint type="free" damping="0.01"/>
-      <geom type="sphere" size="0.03" rgba="0 0 1 0.8" mass="0.2"/>
-      <site name="payload_connection_site" pos="0.0 0.0 0.0"/>
-    </body>
-    <body name="payload_2" pos="-0.7 0.7 0.02">
-      <joint type="free" damping="0.01"/>
-      <geom type="sphere" size="0.03" rgba="0 0 1 0.8" mass="0.2"/>
-      <site name="payload_connection_site_2" pos="0.0 0.0 0.0"/>
-    </body>
+    <!-- AUTO_QUADROTORS_MUJOCO_BODIES -->
+    <!-- AUTO_PAYLOAD_MUJOCO_BODY -->
     <geom name="wall_back" type="box" pos="-3 0 1.5" size="0.05 2 1.5" rgba="0.8 0.8 0.8 0.2"/>
     <geom name="wall_front" type="box" pos="8 0 1.5" size="0.05 2 1.5" rgba="0.8 0.8 0.8 0.2"/>
@@ -70,26 +49,11 @@
   </worldbody>
   <actuator>
-    <xacro:quadrotor_actuators prefix="$(arg quad_name)" />
+    <!-- AUTO_QUADROTORS_MUJOCO_ACTUATORS -->
   </actuator>
   <tendon>
-    <spatial name="rope0" limited="true" range="0 0.71" width=".0005">
-      <site site="$(arg quad_name)_payload_site"/>
-      <site site="payload_connection_site"/>
-    </spatial>
+    <!-- AUTO_QUADROTORS_MUJOCO_TENDONS -->
   </tendon>
   <sensor>
-    <xacro:quadrotor_physical_sensors prefix="$(arg quad_name)" />
-    <xacro:quadrotor_sensor_plugins prefix="$(arg quad_name)" />
-    <plugin name="payload_odom" plugin="MujocoRosUtils::OdometryPublisher" objtype="xbody" objname="payload">
-      <config key="publish_rate" value="100"/>
-      <config key="topic_prefix" value="$(arg quad_name)"/>
-    </plugin>
-    <tendonlimitfrc tendon="rope0"/>
-    <plugin name="rope0_tension_pub" plugin="MujocoRosUtils::TensionPublisher">
-      <config key="tendon_name" value="rope0"/>
-      <config key="topic_prefix" value="$(arg quad_name)"/>
-      <config key="frame_id" value="payload_connection_site"/>
-      <config key="publish_rate" value="100"/>
-    </plugin>
+    <!-- AUTO_QUADROTORS_MUJOCO_SENSORS -->
   </sensor>
 </mujoco>
