Commit message: update macro for lidar

File: model/quadrotor_acro_macro.xml.xacro (robot description, xacro)
@@ -4,5 +4,5 @@
     <mesh name="quadrotor_visual_mesh" file="raxl_assembly.obj" scale="0.001 0.001 0.001" />
   </xacro:macro>
-  <xacro:macro name="quadrotor_body" params="prefix pos euler:='0 0 0' mesh_pos:='-0.17 -0.16 -0.1' mesh_euler:='0 1.57 1.57079632679' primitive_alpha:='0'">
+  <xacro:macro name="quadrotor_body" params="prefix pos euler:='0 0 0' mesh_pos:='-0.17 -0.16 -0.1' mesh_euler:='0 1.57 1.57079632679' primitive_alpha:='0' include_lidar:='false'">
     <body name="${prefix}" pos="${pos}" euler="${euler}">
       <joint name="${prefix}" type="free" damping="0.001" armature="0" pos="0 0 0"/>
@@ -14,4 +14,9 @@
             solref=".5e-4" solimp="0.9 0.99 1e-4" fluidshape="ellipsoid" fluidcoef="3.0 1.0 2.0 1.0 1.0"/>
       <site name="${prefix}_imu" pos="0 0 0"/>
+      <xacro:if value="${include_lidar}">
+        <geom name="${prefix}_lidar_visual" type="box" pos="0 0 0.03" size="0.025 0.018 0.012"
+              rgba="0.0 0.4 1.0 ${primitive_alpha}" contype="0" conaffinity="0" density="0"/>
+        <site name="${prefix}_lidar" type="sphere" pos="0 0 0.03" size="0.01" rgba="0 0.8 1 ${primitive_alpha}"/>
+      </xacro:if>
       <geom name="${prefix}_a00" type="box" pos=".071 0.071 0.0" size="0.05 0.01 0.0025" quat=".924 0 0 0.383" rgba="1 0.5 0 ${primitive_alpha}" mass=".035"
             solref=".5e-4" solimp="0.9 0.99 1e-4" fluidshape="ellipsoid" fluidcoef="3.0 1.0 2.0 1.0 1.0"/>
@@ -109,3 +114,21 @@
     </plugin>
   </xacro:macro>
+  <xacro:macro name="quadrotor_lidar_plugin" params="prefix">
+    <plugin name="${prefix}_lidar_pub" plugin="MujocoRosUtils::LidarPublisher">
+      <config key="site_name" value="${prefix}_lidar"/>
+      <config key="frame_id" value="${prefix}_lidar"/>
+      <config key="topic_prefix" value="${prefix}"/>
+      <config key="topic_name" value="lidar/points"/>
+      <config key="publish_rate" value="10"/>
+      <config key="cutoff_dist" value="30"/>
+      <config key="min_range" value="0.05"/>
+      <config key="scan_model" value="vlp16"/>
+      <config key="horizontal_samples" value="1024"/>
+      <config key="bodyexclude" value="${prefix}"/>
+      <config key="geomgroup" value="1 0 0 0 0 0"/>
+      <config key="qos_reliability" value="reliable"/>
+      <config key="publish_tf" value="true"/>
+      <config key="tf_parent_frame" value="world"/>
+    </plugin>
+  </xacro:macro>
 </mujoco>
