Commit message: Parameterize simulation rates and payload dynamics

File: model/quadrotor_acro_macro.xml.xacro (robot description, xacro)
@@ -50,5 +50,5 @@
     <gyro name="${prefix}_gyro" site="${prefix}_imu" />
   </xacro:macro>
-  <xacro:macro name="quadrotor_actuators" params="prefix">
+  <xacro:macro name="quadrotor_actuators" params="prefix control_hz:=240">
     <plugin site="${prefix}_rotor1_site" name="${prefix}_rotor1"
             plugin="MujocoRosUtils::RotorMotor"
@@ -99,11 +99,11 @@
       <config key="allocation_weight_ty" value="20.0"/>
       <config key="allocation_weight_tz" value="5.0"/>
-      <config key="control_hz"   value="400"/>
+      <config key="control_hz"   value="${control_hz}"/>
       <config key="body_name"    value="${prefix}"/>
     </plugin>
   </xacro:macro>
-  <xacro:macro name="quadrotor_sensor_plugins" params="prefix">
+  <xacro:macro name="quadrotor_sensor_plugins" params="prefix odom_hz:=240 imu_hz:=250">
     <plugin name="${prefix}_odom" plugin="MujocoRosUtils::OdometryPublisher" objtype="xbody" objname="${prefix}">
-      <config key="publish_rate" value="240"/>
+      <config key="publish_rate" value="${odom_hz}"/>
     </plugin>
     <plugin name="${prefix}_imu_pub" plugin="MujocoRosUtils::ImuPublisher">
@@ -111,8 +111,8 @@
       <config key="accel_sensor" value="${prefix}_accel"/>
       <config key="gyro_sensor"  value="${prefix}_gyro"/>
-      <config key="publish_rate" value="400"/>
+      <config key="publish_rate" value="${imu_hz}"/>
     </plugin>
   </xacro:macro>
-  <xacro:macro name="quadrotor_lidar_plugin" params="prefix">
+  <xacro:macro name="quadrotor_lidar_plugin" params="prefix lidar_hz:=10">
     <plugin name="${prefix}_lidar_pub" plugin="MujocoRosUtils::LidarPublisher">
       <config key="site_name" value="${prefix}_lidar"/>
@@ -122,5 +122,5 @@
       <config key="message_type" value="livox_custom"/>
       <config key="livox_lidar_id" value="1"/>
-      <config key="publish_rate" value="10"/>
+      <config key="publish_rate" value="${lidar_hz}"/>
       <config key="cutoff_dist" value="15"/>
       <config key="min_range" value="0.1"/>

File: model/scene.xml.xacro (robot description, xacro)
@@ -39,5 +39,7 @@
     <xacro:quadrotor_body prefix="$(arg quad_name)" pos="$(arg init_x) $(arg init_y) $(arg init_z)" euler="$(arg init_roll) $(arg init_pitch) $(arg init_yaw)" />
     <body name="payload" pos="1 0 0.02">
-      <joint type="free" damping="0.001"/>
+      <joint name="payload_x" type="slide" axis="1 0 0" damping="0.1"/>
+      <joint name="payload_y" type="slide" axis="0 1 0" damping="0.1"/>
+      <joint name="payload_z" type="slide" axis="0 0 1" damping="0.1"/>
       <geom type="sphere" size="0.03" rgba="0 0 1 0.8" mass="0.1"/>
       <site name="payload_connection_site" pos="0.0 0.0 0.03"/>

File: model/scene_acro.xml.xacro (robot description, xacro)
@@ -12,7 +12,15 @@
   <xacro:arg name="mesh_euler" default="0 1.57 1.57079632679"/>
   <xacro:arg name="primitive_alpha" default="0.9"/>
+  <xacro:arg name="simulation_timestep" default="0.003"/>
+  <xacro:arg name="imu_hz" default="250"/>
+  <xacro:arg name="odom_hz" default="240"/>
+  <xacro:arg name="control_hz" default="240"/>
+  <xacro:arg name="payload_odom_hz" default="100"/>
+  <xacro:arg name="tension_hz" default="100"/>
+  <xacro:arg name="clock_hz" default="100"/>
+  <xacro:arg name="lidar_hz" default="10"/>
   <xacro:include filename="quadrotor_acro_macro.xml.xacro" />
   <compiler angle="radian" meshdir="$(arg meshdir)"/>
-  <option timestep="0.002" gravity="0 0 -9.81" density="1.225" viscosity="1.8e-05" integrator="RK4" />
+  <option timestep="$(arg simulation_timestep)" gravity="0 0 -9.81" density="1.225" viscosity="1.8e-05" integrator="RK4" />
   <extension>
     <plugin plugin="MujocoRosUtils::WrenchToActuators"/>
@@ -38,5 +46,5 @@
     <plugin plugin="MujocoRosUtils::ClockPublisher">
       <config key="topic_name" value="/clock"/>
-      <config key="publish_rate" value="100"/>
+      <config key="publish_rate" value="$(arg clock_hz)"/>
       <config key="use_sim_time" value="false"/>
     </plugin>
@@ -53,10 +61,14 @@
                           primitive_alpha="$(arg primitive_alpha)" />
     <body name="payload" pos="-0.7 0.0 0.02">
-      <joint type="free" damping="0.01"/>
+      <joint name="payload_x" type="slide" axis="1 0 0" damping="0.1"/>
+      <joint name="payload_y" type="slide" axis="0 1 0" damping="0.1"/>
+      <joint name="payload_z" type="slide" axis="0 0 1" damping="0.1"/>
       <geom type="sphere" size="0.03" rgba="0 0 1 0.8" mass="0.2"/>
       <site name="payload_connection_site" pos="0.0 0.0 0.0"/>
     </body>
     <body name="payload_2" pos="-0.7 0.7 0.02">
-      <joint type="free" damping="0.01"/>
+      <joint name="payload_2_x" type="slide" axis="1 0 0" damping="0.1"/>
+      <joint name="payload_2_y" type="slide" axis="0 1 0" damping="0.1"/>
+      <joint name="payload_2_z" type="slide" axis="0 0 1" damping="0.1"/>
       <geom type="sphere" size="0.03" rgba="0 0 1 0.8" mass="0.2"/>
       <site name="payload_connection_site_2" pos="0.0 0.0 0.0"/>
@@ -71,5 +83,5 @@
   </worldbody>
   <actuator>
-    <xacro:quadrotor_actuators prefix="$(arg quad_name)" />
+    <xacro:quadrotor_actuators prefix="$(arg quad_name)" control_hz="$(arg control_hz)" />
   </actuator>
   <tendon>
@@ -81,7 +93,7 @@
   <sensor>
     <xacro:quadrotor_physical_sensors prefix="$(arg quad_name)" />
-    <xacro:quadrotor_sensor_plugins prefix="$(arg quad_name)" />
+    <xacro:quadrotor_sensor_plugins prefix="$(arg quad_name)" odom_hz="$(arg odom_hz)" imu_hz="$(arg imu_hz)" />
     <plugin name="payload_odom" plugin="MujocoRosUtils::OdometryPublisher" objtype="xbody" objname="payload">
-      <config key="publish_rate" value="240"/>
+      <config key="publish_rate" value="$(arg payload_odom_hz)"/>
       <config key="topic_prefix" value="$(arg quad_name)"/>
     </plugin>
@@ -91,5 +103,5 @@
       <config key="topic_prefix" value="$(arg quad_name)"/>
       <config key="frame_id" value="payload_connection_site"/>
-      <config key="publish_rate" value="240"/>
+      <config key="publish_rate" value="$(arg tension_hz)"/>
     </plugin>
   </sensor>

File: model/scene_acro_gate.xml.xacro (robot description, xacro)
@@ -12,4 +12,12 @@
   <xacro:arg name="mesh_euler" default="0 1.57 1.57079632679"/>
   <xacro:arg name="primitive_alpha" default="0.9"/>
+  <xacro:arg name="simulation_timestep" default="0.003"/>
+  <xacro:arg name="imu_hz" default="250"/>
+  <xacro:arg name="odom_hz" default="240"/>
+  <xacro:arg name="control_hz" default="240"/>
+  <xacro:arg name="payload_odom_hz" default="100"/>
+  <xacro:arg name="tension_hz" default="100"/>
+  <xacro:arg name="clock_hz" default="100"/>
+  <xacro:arg name="lidar_hz" default="10"/>
   <xacro:arg name="gates_collide" default="0"/>
   <xacro:arg name="gate_radius" default="0.42"/>
@@ -18,5 +26,5 @@
   <xacro:include filename="quadrotor_acro_macro.xml.xacro" />
   <compiler angle="radian" meshdir="$(arg meshdir)"/>
-  <option timestep="0.002" gravity="0 0 -9.81" density="1.225" viscosity="1.8e-05" integrator="RK4" />
+  <option timestep="$(arg simulation_timestep)" gravity="0 0 -9.81" density="1.225" viscosity="1.8e-05" integrator="RK4" />
   <extension>
     <plugin plugin="MujocoRosUtils::WrenchToActuators"/>
@@ -63,5 +71,5 @@
     <plugin plugin="MujocoRosUtils::ClockPublisher">
       <config key="topic_name" value="/clock"/>
-      <config key="publish_rate" value="100"/>
+      <config key="publish_rate" value="$(arg clock_hz)"/>
       <config key="use_sim_time" value="false"/>
     </plugin>
@@ -78,10 +86,14 @@
                           primitive_alpha="$(arg primitive_alpha)" />
     <body name="payload" pos="-0.0 0.0 0.7">
-      <joint type="free" damping="0.01"/>
+      <joint name="payload_x" type="slide" axis="1 0 0" damping="0.1"/>
+      <joint name="payload_y" type="slide" axis="0 1 0" damping="0.1"/>
+      <joint name="payload_z" type="slide" axis="0 0 1" damping="0.1"/>
       <geom type="sphere" size="0.03" rgba="0 0 1 0.8" mass="0.2"/>
       <site name="payload_connection_site" pos="0.0 0.0 0.0"/>
     </body>
     <body name="payload_2" pos="-0.7 0.7 0.02">
-      <joint type="free" damping="0.01"/>
+      <joint name="payload_2_x" type="slide" axis="1 0 0" damping="0.1"/>
+      <joint name="payload_2_y" type="slide" axis="0 1 0" damping="0.1"/>
+      <joint name="payload_2_z" type="slide" axis="0 0 1" damping="0.1"/>
       <geom type="sphere" size="0.03" rgba="0 0 1 0.8" mass="0.2"/>
       <site name="payload_connection_site_2" pos="0.0 0.0 0.0"/>
@@ -100,5 +112,5 @@
   </worldbody>
   <actuator>
-    <xacro:quadrotor_actuators prefix="$(arg quad_name)" />
+    <xacro:quadrotor_actuators prefix="$(arg quad_name)" control_hz="$(arg control_hz)" />
   </actuator>
   <tendon>
@@ -110,7 +122,7 @@
   <sensor>
     <xacro:quadrotor_physical_sensors prefix="$(arg quad_name)" />
-    <xacro:quadrotor_sensor_plugins prefix="$(arg quad_name)" />
+    <xacro:quadrotor_sensor_plugins prefix="$(arg quad_name)" odom_hz="$(arg odom_hz)" imu_hz="$(arg imu_hz)" />
     <plugin name="payload_odom" plugin="MujocoRosUtils::OdometryPublisher" objtype="xbody" objname="payload">
-      <config key="publish_rate" value="240"/>
+      <config key="publish_rate" value="$(arg payload_odom_hz)"/>
       <config key="topic_prefix" value="$(arg quad_name)"/>
     </plugin>
@@ -120,5 +132,5 @@
       <config key="topic_prefix" value="$(arg quad_name)"/>
       <config key="frame_id" value="payload_connection_site"/>
-      <config key="publish_rate" value="240"/>
+      <config key="publish_rate" value="$(arg tension_hz)"/>
     </plugin>
   </sensor>

File: model/scene_acro_humanoid.xml.xacro (robot description, xacro)
@@ -39,5 +39,7 @@
     <xacro:g1_humanoid_body prefix="g1" pos="3 0 0.793" euler="0 0 0"/>
     <body name="payload" pos="0.8 0 0.02">
-      <joint type="free" damping="0.01"/>
+      <joint name="payload_x" type="slide" axis="1 0 0" damping="0.1"/>
+      <joint name="payload_y" type="slide" axis="0 1 0" damping="0.1"/>
+      <joint name="payload_z" type="slide" axis="0 0 1" damping="0.1"/>
       <geom type="sphere" size="0.03" rgba="0 0 1 0.8" mass="0.1128"/>
       <site name="payload_connection_site" pos="0.0 0.0 0.03"/>

File: model/scene_acro_lidar.xml.xacro (robot description, xacro)
@@ -12,7 +12,15 @@
   <xacro:arg name="mesh_euler" default="0 1.57 1.57079632679"/>
   <xacro:arg name="primitive_alpha" default="0.9"/>
+  <xacro:arg name="simulation_timestep" default="0.003"/>
+  <xacro:arg name="imu_hz" default="250"/>
+  <xacro:arg name="odom_hz" default="240"/>
+  <xacro:arg name="control_hz" default="240"/>
+  <xacro:arg name="payload_odom_hz" default="100"/>
+  <xacro:arg name="tension_hz" default="100"/>
+  <xacro:arg name="clock_hz" default="100"/>
+  <xacro:arg name="lidar_hz" default="10"/>
   <xacro:include filename="quadrotor_acro_macro.xml.xacro" />
   <compiler angle="radian" meshdir="$(arg meshdir)"/>
-  <option timestep="0.002" gravity="0 0 -9.81" density="1.225" viscosity="1.8e-05" integrator="RK4" />
+  <option timestep="$(arg simulation_timestep)" gravity="0 0 -9.81" density="1.225" viscosity="1.8e-05" integrator="RK4" />
   <extension>
     <plugin plugin="MujocoRosUtils::WrenchToActuators"/>
@@ -42,5 +50,5 @@
     <plugin plugin="MujocoRosUtils::ClockPublisher">
       <config key="topic_name" value="/clock"/>
-      <config key="publish_rate" value="100"/>
+      <config key="publish_rate" value="$(arg clock_hz)"/>
       <config key="use_sim_time" value="false"/>
     </plugin>
@@ -65,10 +73,14 @@
                           include_lidar="true" />
     <body name="payload" pos="-0.7 0.0 0.02">
-      <joint type="free" damping="0.01"/>
+      <joint name="payload_x" type="slide" axis="1 0 0" damping="0.1"/>
+      <joint name="payload_y" type="slide" axis="0 1 0" damping="0.1"/>
+      <joint name="payload_z" type="slide" axis="0 0 1" damping="0.1"/>
       <geom type="sphere" size="0.03" rgba="0 0 1 0.8" mass="0.2"/>
       <site name="payload_connection_site" pos="0.0 0.0 0.0"/>
     </body>
     <body name="payload_2" pos="-0.7 0.7 0.02">
-      <joint type="free" damping="0.01"/>
+      <joint name="payload_2_x" type="slide" axis="1 0 0" damping="0.1"/>
+      <joint name="payload_2_y" type="slide" axis="0 1 0" damping="0.1"/>
+      <joint name="payload_2_z" type="slide" axis="0 0 1" damping="0.1"/>
       <geom type="sphere" size="0.03" rgba="0 0 1 0.8" mass="0.2"/>
       <site name="payload_connection_site_2" pos="0.0 0.0 0.0"/>
@@ -83,5 +95,5 @@
   </worldbody>
   <actuator>
-    <xacro:quadrotor_actuators prefix="$(arg quad_name)" />
+    <xacro:quadrotor_actuators prefix="$(arg quad_name)" control_hz="$(arg control_hz)" />
   </actuator>
   <tendon>
@@ -93,8 +105,8 @@
   <sensor>
     <xacro:quadrotor_physical_sensors prefix="$(arg quad_name)" />
-    <xacro:quadrotor_sensor_plugins prefix="$(arg quad_name)" />
-    <xacro:quadrotor_lidar_plugin prefix="$(arg quad_name)" />
+    <xacro:quadrotor_sensor_plugins prefix="$(arg quad_name)" odom_hz="$(arg odom_hz)" imu_hz="$(arg imu_hz)" />
+    <xacro:quadrotor_lidar_plugin prefix="$(arg quad_name)" lidar_hz="$(arg lidar_hz)" />
     <plugin name="payload_odom" plugin="MujocoRosUtils::OdometryPublisher" objtype="xbody" objname="payload">
-      <config key="publish_rate" value="240"/>
+      <config key="publish_rate" value="$(arg payload_odom_hz)"/>
       <config key="topic_prefix" value="$(arg quad_name)"/>
     </plugin>
@@ -104,5 +116,5 @@
       <config key="topic_prefix" value="$(arg quad_name)"/>
       <config key="frame_id" value="payload_connection_site"/>
-      <config key="publish_rate" value="240"/>
+      <config key="publish_rate" value="$(arg tension_hz)"/>
     </plugin>
   </sensor>

File: model/scene_acro_multiple.xml.xacro (robot description, xacro)
@@ -46,5 +46,7 @@
     <xacro:quadrotor_body prefix="$(arg quad_name_2)" pos="$(arg init_x_2) $(arg init_y_2) $(arg init_z_2)" euler="$(arg init_roll_2) $(arg init_pitch_2) $(arg init_yaw_2)" />
     <body name="payload" pos="0.3 0.3 1.0">
-      <joint type="free" damping="0.01"/>
+      <joint name="payload_x" type="slide" axis="1 0 0" damping="0.1"/>
+      <joint name="payload_y" type="slide" axis="0 1 0" damping="0.1"/>
+      <joint name="payload_z" type="slide" axis="0 0 1" damping="0.1"/>
       <geom type="sphere" size="0.03" rgba="0 0 1 0.8" mass="0.1128"/>
       <site name="payload_connection_site" pos="0.0 0.0 0.03"/>

File: model/scene_acro_payload.xml.xacro (robot description, xacro)
@@ -12,7 +12,15 @@
   <xacro:arg name="mesh_euler" default="0 1.57 1.57079632679"/>
   <xacro:arg name="primitive_alpha" default="0.9"/>
+  <xacro:arg name="simulation_timestep" default="0.003"/>
+  <xacro:arg name="imu_hz" default="250"/>
+  <xacro:arg name="odom_hz" default="240"/>
+  <xacro:arg name="control_hz" default="240"/>
+  <xacro:arg name="payload_odom_hz" default="100"/>
+  <xacro:arg name="tension_hz" default="100"/>
+  <xacro:arg name="clock_hz" default="100"/>
+  <xacro:arg name="lidar_hz" default="10"/>
   <xacro:include filename="quadrotor_acro_macro.xml.xacro" />
   <compiler angle="radian" meshdir="$(arg meshdir)"/>
-  <option timestep="0.002" gravity="0 0 -9.81" density="1.225" viscosity="1.8e-05" integrator="RK4" />
+  <option timestep="$(arg simulation_timestep)" gravity="0 0 -9.81" density="1.225" viscosity="1.8e-05" integrator="RK4" />
   <extension>
     <plugin plugin="MujocoRosUtils::WrenchToActuators"/>
@@ -38,5 +46,5 @@
     <plugin plugin="MujocoRosUtils::ClockPublisher">
       <config key="topic_name" value="/clock"/>
-      <config key="publish_rate" value="100"/>
+      <config key="publish_rate" value="$(arg clock_hz)"/>
       <config key="use_sim_time" value="false"/>
     </plugin>
@@ -53,10 +61,14 @@
                           primitive_alpha="$(arg primitive_alpha)" />
     <body name="payload" pos="-0.7 0.0 0.02">
-      <joint type="free" damping="0.01"/>
+      <joint name="payload_x" type="slide" axis="1 0 0" damping="0.1"/>
+      <joint name="payload_y" type="slide" axis="0 1 0" damping="0.1"/>
+      <joint name="payload_z" type="slide" axis="0 0 1" damping="0.1"/>
       <geom type="sphere" size="0.03" rgba="0 0 1 0.8" mass="0.2"/>
       <site name="payload_connection_site" pos="0.0 0.0 0.0"/>
     </body>
     <body name="payload_2" pos="-0.7 0.7 0.02">
-      <joint type="free" damping="0.01"/>
+      <joint name="payload_2_x" type="slide" axis="1 0 0" damping="0.1"/>
+      <joint name="payload_2_y" type="slide" axis="0 1 0" damping="0.1"/>
+      <joint name="payload_2_z" type="slide" axis="0 0 1" damping="0.1"/>
       <geom type="sphere" size="0.03" rgba="0 0 1 0.8" mass="0.2"/>
       <site name="payload_connection_site_2" pos="0.0 0.0 0.0"/>
@@ -71,5 +83,5 @@
   </worldbody>
   <actuator>
-    <xacro:quadrotor_actuators prefix="$(arg quad_name)" />
+    <xacro:quadrotor_actuators prefix="$(arg quad_name)" control_hz="$(arg control_hz)" />
   </actuator>
   <tendon>
@@ -81,7 +93,7 @@
   <sensor>
     <xacro:quadrotor_physical_sensors prefix="$(arg quad_name)" />
-    <xacro:quadrotor_sensor_plugins prefix="$(arg quad_name)" />
+    <xacro:quadrotor_sensor_plugins prefix="$(arg quad_name)" odom_hz="$(arg odom_hz)" imu_hz="$(arg imu_hz)" />
     <plugin name="payload_odom" plugin="MujocoRosUtils::OdometryPublisher" objtype="xbody" objname="payload">
-      <config key="publish_rate" value="240"/>
+      <config key="publish_rate" value="$(arg payload_odom_hz)"/>
       <config key="topic_prefix" value="$(arg quad_name)"/>
     </plugin>
@@ -91,5 +103,5 @@
       <config key="topic_prefix" value="$(arg quad_name)"/>
       <config key="frame_id" value="payload_connection_site"/>
-      <config key="publish_rate" value="240"/>
+      <config key="publish_rate" value="$(arg tension_hz)"/>
     </plugin>
   </sensor>

File: model/scene_acro_payload_lidar.xml.xacro (robot description, xacro)
@@ -12,7 +12,15 @@
   <xacro:arg name="mesh_euler" default="0 1.57 1.57079632679"/>
   <xacro:arg name="primitive_alpha" default="0.9"/>
+  <xacro:arg name="simulation_timestep" default="0.003"/>
+  <xacro:arg name="imu_hz" default="250"/>
+  <xacro:arg name="odom_hz" default="240"/>
+  <xacro:arg name="control_hz" default="240"/>
+  <xacro:arg name="payload_odom_hz" default="100"/>
+  <xacro:arg name="tension_hz" default="100"/>
+  <xacro:arg name="clock_hz" default="100"/>
+  <xacro:arg name="lidar_hz" default="10"/>
   <xacro:include filename="quadrotor_acro_macro.xml.xacro" />
   <compiler angle="radian" meshdir="$(arg meshdir)"/>
-  <option timestep="0.002" gravity="0 0 -9.81" density="1.225" viscosity="1.8e-05" integrator="RK4" />
+  <option timestep="$(arg simulation_timestep)" gravity="0 0 -9.81" density="1.225" viscosity="1.8e-05" integrator="RK4" />
   <extension>
     <plugin plugin="MujocoRosUtils::WrenchToActuators"/>
@@ -42,5 +50,5 @@
     <plugin plugin="MujocoRosUtils::ClockPublisher">
       <config key="topic_name" value="/clock"/>
-      <config key="publish_rate" value="100"/>
+      <config key="publish_rate" value="$(arg clock_hz)"/>
       <config key="use_sim_time" value="false"/>
     </plugin>
@@ -65,10 +73,14 @@
                           include_lidar="true" />
     <body name="payload" pos="-0.7 0.0 0.02">
-      <joint type="free" damping="0.01"/>
+      <joint name="payload_x" type="slide" axis="1 0 0" damping="0.1"/>
+      <joint name="payload_y" type="slide" axis="0 1 0" damping="0.1"/>
+      <joint name="payload_z" type="slide" axis="0 0 1" damping="0.1"/>
       <geom type="sphere" size="0.03" rgba="0 0 1 0.8" mass="0.2"/>
       <site name="payload_connection_site" pos="0.0 0.0 0.0"/>
     </body>
     <body name="payload_2" pos="-0.7 0.7 0.02">
-      <joint type="free" damping="0.01"/>
+      <joint name="payload_2_x" type="slide" axis="1 0 0" damping="0.1"/>
+      <joint name="payload_2_y" type="slide" axis="0 1 0" damping="0.1"/>
+      <joint name="payload_2_z" type="slide" axis="0 0 1" damping="0.1"/>
       <geom type="sphere" size="0.03" rgba="0 0 1 0.8" mass="0.2"/>
       <site name="payload_connection_site_2" pos="0.0 0.0 0.0"/>
@@ -83,5 +95,5 @@
   </worldbody>
   <actuator>
-    <xacro:quadrotor_actuators prefix="$(arg quad_name)" />
+    <xacro:quadrotor_actuators prefix="$(arg quad_name)" control_hz="$(arg control_hz)" />
   </actuator>
   <tendon>
@@ -93,8 +105,8 @@
   <sensor>
     <xacro:quadrotor_physical_sensors prefix="$(arg quad_name)" />
-    <xacro:quadrotor_sensor_plugins prefix="$(arg quad_name)" />
-    <xacro:quadrotor_lidar_plugin prefix="$(arg quad_name)" />
+    <xacro:quadrotor_sensor_plugins prefix="$(arg quad_name)" odom_hz="$(arg odom_hz)" imu_hz="$(arg imu_hz)" />
+    <xacro:quadrotor_lidar_plugin prefix="$(arg quad_name)" lidar_hz="$(arg lidar_hz)" />
     <plugin name="payload_odom" plugin="MujocoRosUtils::OdometryPublisher" objtype="xbody" objname="payload">
-      <config key="publish_rate" value="240"/>
+      <config key="publish_rate" value="$(arg payload_odom_hz)"/>
       <config key="topic_prefix" value="$(arg quad_name)"/>
     </plugin>
@@ -104,5 +116,5 @@
       <config key="topic_prefix" value="$(arg quad_name)"/>
       <config key="frame_id" value="payload_connection_site"/>
-      <config key="publish_rate" value="240"/>
+      <config key="publish_rate" value="$(arg tension_hz)"/>
     </plugin>
   </sensor>

File: model/scene_acro_point_mass_multiple.xml.xacro (robot description, xacro)
@@ -5,7 +5,9 @@
   <xacro:arg name="mesh_euler" default="0 1.57 1.57079632679"/>
   <xacro:arg name="primitive_alpha" default="0.8"/>
+  <xacro:arg name="simulation_timestep" default="0.003"/>
+  <xacro:arg name="clock_hz" default="100"/>
   <xacro:include filename="quadrotor_acro_macro.xml.xacro" />
   <compiler angle="radian" meshdir="$(arg meshdir)"/>
-  <option timestep="0.002" gravity="0 0 -9.81" density="1.225" viscosity="1.8e-05" integrator="RK4" />
+  <option timestep="$(arg simulation_timestep)" gravity="0 0 -9.81" density="1.225" viscosity="1.8e-05" integrator="RK4" />
   <extension>
     <plugin plugin="MujocoRosUtils::WrenchToActuators"/>
@@ -31,5 +33,5 @@
     <plugin plugin="MujocoRosUtils::ClockPublisher">
       <config key="topic_name" value="/clock"/>
-      <config key="publish_rate" value="100"/>
+      <config key="publish_rate" value="$(arg clock_hz)"/>
       <config key="use_sim_time" value="false"/>
     </plugin>
