Commit message: Parameterize simulation rates and payload dynamics

File: model/scene_acro_point_mass_multiple_lidar.xml.xacro (robot description, xacro)
@@ -5,7 +5,9 @@
   <xacro:arg name="mesh_euler" default="0 1.57 1.57079632679"/>
   <xacro:arg name="primitive_alpha" default="0.8"/>
+  <xacro:arg name="simulation_timestep" default="0.003"/>
+  <xacro:arg name="clock_hz" default="100"/>
   <xacro:include filename="quadrotor_acro_macro.xml.xacro" />
   <compiler angle="radian" meshdir="$(arg meshdir)"/>
-  <option timestep="0.002" gravity="0 0 -9.81" density="1.225" viscosity="1.8e-05" integrator="RK4" />
+  <option timestep="$(arg simulation_timestep)" gravity="0 0 -9.81" density="1.225" viscosity="1.8e-05" integrator="RK4" />
   <extension>
     <plugin plugin="MujocoRosUtils::WrenchToActuators"/>
@@ -35,5 +37,5 @@
     <plugin plugin="MujocoRosUtils::ClockPublisher">
       <config key="topic_name" value="/clock"/>
-      <config key="publish_rate" value="100"/>
+      <config key="publish_rate" value="$(arg clock_hz)"/>
       <config key="use_sim_time" value="false"/>
     </plugin>

File: model/scene_inertial_force_sphere.xml.xacro (robot description, xacro)
@@ -15,5 +15,5 @@
   <xacro:arg name="payload_radius" default="0.03"/>
   <xacro:arg name="payload_mass" default="0.2"/>
-  <xacro:arg name="payload_damping" default="0.002"/>
+  <xacro:arg name="payload_damping" default="0.1"/>
   <xacro:arg name="cable_length" default="0.71"/>
   <xacro:arg name="publish_rate" default="240"/>

File: model/scene_lowlevel.xml.xacro (robot description, xacro)
@@ -37,5 +37,7 @@
     <xacro:quadrotor_body prefix="$(arg quad_name)" pos="$(arg init_x) $(arg init_y) $(arg init_z)" euler="$(arg init_roll) $(arg init_pitch) $(arg init_yaw)" />
     <body name="payload" pos="0.6 0 0.02">
-      <joint type="free" damping="0.001"/>
+      <joint name="payload_x" type="slide" axis="1 0 0" damping="0.1"/>
+      <joint name="payload_y" type="slide" axis="0 1 0" damping="0.1"/>
+      <joint name="payload_z" type="slide" axis="0 0 1" damping="0.1"/>
       <geom type="sphere" size="0.03" rgba="0 0 1 0.8" mass="0.1128"/>
       <site name="payload_connection_site" pos="0.0 0.0 0.03"/>

File: model/scene_so3.xml.xacro (robot description, xacro)
@@ -38,5 +38,7 @@
     <xacro:quadrotor_body prefix="$(arg quad_name)" pos="$(arg init_x) $(arg init_y) $(arg init_z)" euler="$(arg init_roll) $(arg init_pitch) $(arg init_yaw)" />
     <body name="payload" pos="0.6 0 0.02">
-      <joint type="free" damping="0.001"/>
+      <joint name="payload_x" type="slide" axis="1 0 0" damping="0.1"/>
+      <joint name="payload_y" type="slide" axis="0 1 0" damping="0.1"/>
+      <joint name="payload_z" type="slide" axis="0 0 1" damping="0.1"/>
       <geom type="sphere" size="0.03" rgba="0 0 1 0.8" mass="0.1128"/>
       <site name="payload_connection_site" pos="0.0 0.0 0.03"/>

Commit message: Tune simulation timestep and sensor rates

File: model/quadrotor_acro_macro.xml.xacro (robot description, xacro)
@@ -103,5 +103,5 @@
     </plugin>
   </xacro:macro>
-  <xacro:macro name="quadrotor_sensor_plugins" params="prefix odom_hz:=240 imu_hz:=250">
+  <xacro:macro name="quadrotor_sensor_plugins" params="prefix odom_hz:=240 imu_hz:=350">
     <plugin name="${prefix}_odom" plugin="MujocoRosUtils::OdometryPublisher" objtype="xbody" objname="${prefix}">
       <config key="publish_rate" value="${odom_hz}"/>

File: model/scene.xml.xacro (robot description, xacro)
@@ -12,5 +12,5 @@
   <xacro:include filename="quadrotor_lowlevel_macro.xml.xacro" />
   <compiler angle="radian"/>
-  <option timestep="0.003" gravity="0 0 -9.81" density="1.225" viscosity="1.8e-05" integrator="RK4" />
+  <option timestep="0.0025" gravity="0 0 -9.81" density="1.225" viscosity="1.8e-05" integrator="RK4" />
   <extension>
     <plugin plugin="MujocoRosUtils::WrenchToActuators"/>

File: model/scene_acro.xml.xacro (robot description, xacro)
@@ -12,9 +12,9 @@
   <xacro:arg name="mesh_euler" default="0 1.57 1.57079632679"/>
   <xacro:arg name="primitive_alpha" default="0.9"/>
-  <xacro:arg name="simulation_timestep" default="0.003"/>
-  <xacro:arg name="imu_hz" default="250"/>
+  <xacro:arg name="simulation_timestep" default="0.0025"/>
+  <xacro:arg name="imu_hz" default="350"/>
   <xacro:arg name="odom_hz" default="240"/>
   <xacro:arg name="control_hz" default="240"/>
-  <xacro:arg name="payload_odom_hz" default="100"/>
+  <xacro:arg name="payload_odom_hz" default="240"/>
   <xacro:arg name="tension_hz" default="100"/>
   <xacro:arg name="clock_hz" default="100"/>

File: model/scene_acro_gate.xml.xacro (robot description, xacro)
@@ -12,9 +12,9 @@
   <xacro:arg name="mesh_euler" default="0 1.57 1.57079632679"/>
   <xacro:arg name="primitive_alpha" default="0.9"/>
-  <xacro:arg name="simulation_timestep" default="0.003"/>
-  <xacro:arg name="imu_hz" default="250"/>
+  <xacro:arg name="simulation_timestep" default="0.0025"/>
+  <xacro:arg name="imu_hz" default="350"/>
   <xacro:arg name="odom_hz" default="240"/>
   <xacro:arg name="control_hz" default="240"/>
-  <xacro:arg name="payload_odom_hz" default="100"/>
+  <xacro:arg name="payload_odom_hz" default="240"/>
   <xacro:arg name="tension_hz" default="100"/>
   <xacro:arg name="clock_hz" default="100"/>

File: model/scene_acro_humanoid.xml.xacro (robot description, xacro)
@@ -11,5 +11,5 @@
   <xacro:include filename="humanoid_macro.xml.xacro"/>
   <compiler angle="radian" meshdir="/home/fer/payload_transportation_ws/src/acp_mujoco_simulator/model/humanoid_resource/meshes"/>
-  <option timestep="0.003" gravity="0 0 -9.81" density="1.225" viscosity="1.8e-05" integrator="RK4" />
+  <option timestep="0.0025" gravity="0 0 -9.81" density="1.225" viscosity="1.8e-05" integrator="RK4" />
   <extension>
     <plugin plugin="MujocoRosUtils::WrenchToActuators"/>

File: model/scene_acro_lidar.xml.xacro (robot description, xacro)
@@ -12,9 +12,9 @@
   <xacro:arg name="mesh_euler" default="0 1.57 1.57079632679"/>
   <xacro:arg name="primitive_alpha" default="0.9"/>
-  <xacro:arg name="simulation_timestep" default="0.003"/>
-  <xacro:arg name="imu_hz" default="250"/>
+  <xacro:arg name="simulation_timestep" default="0.0025"/>
+  <xacro:arg name="imu_hz" default="350"/>
   <xacro:arg name="odom_hz" default="240"/>
   <xacro:arg name="control_hz" default="240"/>
-  <xacro:arg name="payload_odom_hz" default="100"/>
+  <xacro:arg name="payload_odom_hz" default="240"/>
   <xacro:arg name="tension_hz" default="100"/>
   <xacro:arg name="clock_hz" default="100"/>

File: model/scene_acro_multiple.xml.xacro (robot description, xacro)
@@ -17,5 +17,5 @@
   <xacro:include filename="quadrotor_acro_macro.xml.xacro" />
   <compiler angle="radian"/>
-  <option timestep="0.003" gravity="0 0 -9.81" density="1.225" viscosity="1.8e-05" integrator="RK4">
+  <option timestep="0.0025" gravity="0 0 -9.81" density="1.225" viscosity="1.8e-05" integrator="RK4">
     <flag contact="disable"/>
   </option>

File: model/scene_acro_payload.xml.xacro (robot description, xacro)
@@ -12,9 +12,9 @@
   <xacro:arg name="mesh_euler" default="0 1.57 1.57079632679"/>
   <xacro:arg name="primitive_alpha" default="0.9"/>
-  <xacro:arg name="simulation_timestep" default="0.003"/>
-  <xacro:arg name="imu_hz" default="250"/>
+  <xacro:arg name="simulation_timestep" default="0.0025"/>
+  <xacro:arg name="imu_hz" default="350"/>
   <xacro:arg name="odom_hz" default="240"/>
   <xacro:arg name="control_hz" default="240"/>
-  <xacro:arg name="payload_odom_hz" default="100"/>
+  <xacro:arg name="payload_odom_hz" default="240"/>
   <xacro:arg name="tension_hz" default="100"/>
   <xacro:arg name="clock_hz" default="100"/>

File: model/scene_acro_payload_lidar.xml.xacro (robot description, xacro)
@@ -12,9 +12,9 @@
   <xacro:arg name="mesh_euler" default="0 1.57 1.57079632679"/>
   <xacro:arg name="primitive_alpha" default="0.9"/>
-  <xacro:arg name="simulation_timestep" default="0.003"/>
-  <xacro:arg name="imu_hz" default="250"/>
+  <xacro:arg name="simulation_timestep" default="0.0025"/>
+  <xacro:arg name="imu_hz" default="350"/>
   <xacro:arg name="odom_hz" default="240"/>
   <xacro:arg name="control_hz" default="240"/>
-  <xacro:arg name="payload_odom_hz" default="100"/>
+  <xacro:arg name="payload_odom_hz" default="240"/>
   <xacro:arg name="tension_hz" default="100"/>
   <xacro:arg name="clock_hz" default="100"/>

File: model/scene_acro_point_mass_multiple.xml.xacro (robot description, xacro)
@@ -5,5 +5,5 @@
   <xacro:arg name="mesh_euler" default="0 1.57 1.57079632679"/>
   <xacro:arg name="primitive_alpha" default="0.8"/>
-  <xacro:arg name="simulation_timestep" default="0.003"/>
+  <xacro:arg name="simulation_timestep" default="0.0025"/>
   <xacro:arg name="clock_hz" default="100"/>
   <xacro:include filename="quadrotor_acro_macro.xml.xacro" />

File: model/scene_acro_point_mass_multiple_lidar.xml.xacro (robot description, xacro)
@@ -5,5 +5,5 @@
   <xacro:arg name="mesh_euler" default="0 1.57 1.57079632679"/>
   <xacro:arg name="primitive_alpha" default="0.8"/>
-  <xacro:arg name="simulation_timestep" default="0.003"/>
+  <xacro:arg name="simulation_timestep" default="0.0025"/>
   <xacro:arg name="clock_hz" default="100"/>
   <xacro:include filename="quadrotor_acro_macro.xml.xacro" />

File: model/scene_inertial_force_sphere.xml.xacro (robot description, xacro)
@@ -20,5 +20,5 @@
   <xacro:arg name="use_sim_time" default="false"/>
   <compiler angle="radian"/>
-  <option timestep="0.002" gravity="0 0 -9.81" density="1.225" viscosity="1.8e-05" integrator="RK4"/>
+  <option timestep="0.0025" gravity="0 0 -9.81" density="1.225" viscosity="1.8e-05" integrator="RK4"/>
   <extension>
     <plugin plugin="MujocoRosUtils::ActuatorCommand"/>

File: model/scene_lowlevel.xml.xacro (robot description, xacro)
@@ -10,5 +10,5 @@
   <xacro:include filename="quadrotor_lowlevel_macro.xml.xacro" />
   <compiler angle="radian"/>
-  <option timestep="0.002" gravity="0 0 -9.81" density="1.225" viscosity="1.8e-05" integrator="RK4" />
+  <option timestep="0.0025" gravity="0 0 -9.81" density="1.225" viscosity="1.8e-05" integrator="RK4" />
   <extension>
     <plugin plugin="MujocoRosUtils::WrenchToActuators"/>

File: model/scene_so3.xml.xacro (robot description, xacro)
@@ -10,5 +10,5 @@
   <xacro:include filename="quadrotor_so3_macro.xml.xacro" />
   <compiler angle="radian"/>
-  <option timestep="0.003" gravity="0 0 -9.81" density="1.225" viscosity="1.8e-05" integrator="RK4" />
+  <option timestep="0.0025" gravity="0 0 -9.81" density="1.225" viscosity="1.8e-05" integrator="RK4" />
   <extension>
     <plugin plugin="MujocoRosUtils::WrenchToActuators"/>
