Commit message: Format tools and refine simulation models

File: model/scene_acro_lidar.xml.xacro (robot description, xacro)
@@ -76,5 +76,5 @@
       <joint name="payload_y" type="slide" axis="0 1 0" damping="0.2"/>
       <joint name="payload_z" type="slide" axis="0 0 1" damping="0.2"/>
-      <geom type="sphere" size="0.03" rgba="0 0 1 0.8" mass="0.2"/>
+      <geom type="sphere" size="0.035" rgba="0 0 1 0.8" mass="0.2"/>
       <site name="payload_connection_site" pos="0.0 0.0 0.0"/>
     </body>
@@ -83,5 +83,5 @@
       <joint name="payload_2_y" type="slide" axis="0 1 0" damping="0.2"/>
       <joint name="payload_2_z" type="slide" axis="0 0 1" damping="0.2"/>
-      <geom type="sphere" size="0.03" rgba="0 0 1 0.8" mass="0.2"/>
+      <geom type="sphere" size="0.035" rgba="0 0 1 0.8" mass="0.2"/>
       <site name="payload_connection_site_2" pos="0.0 0.0 0.0"/>
     </body>

File: model/scene_acro_multiple.xml.xacro (robot description, xacro)
@@ -49,6 +49,6 @@
       <joint name="payload_y" type="slide" axis="0 1 0" damping="0.2"/>
       <joint name="payload_z" type="slide" axis="0 0 1" damping="0.2"/>
-      <geom type="sphere" size="0.03" rgba="0 0 1 0.8" mass="0.1128"/>
-      <site name="payload_connection_site" pos="0.0 0.0 0.03"/>
+      <geom type="sphere" size="0.035" rgba="0 0 1 0.8" mass="0.1128"/>
+      <site name="payload_connection_site" pos="0.0 0.0 0.035"/>
     </body>
     <geom name="origin_x" type="cylinder" fromto="0 0 0.01 0.5 0 0.01" size="0.01" rgba="1 0 0 0.1" contype="0" conaffinity="0" group="1"/>

File: model/scene_acro_payload.xml.xacro (robot description, xacro)
@@ -64,5 +64,5 @@
       <joint name="payload_y" type="slide" axis="0 1 0" damping="0.2"/>
       <joint name="payload_z" type="slide" axis="0 0 1" damping="0.2"/>
-      <geom type="sphere" size="0.03" rgba="0 0 1 0.8" mass="0.2"/>
+      <geom type="sphere" size="0.035" rgba="0 0 1 0.8" mass="0.2"/>
       <site name="payload_connection_site" pos="0.0 0.0 0.0"/>
     </body>
@@ -71,5 +71,5 @@
       <joint name="payload_2_y" type="slide" axis="0 1 0" damping="0.2"/>
       <joint name="payload_2_z" type="slide" axis="0 0 1" damping="0.2"/>
-      <geom type="sphere" size="0.03" rgba="0 0 1 0.8" mass="0.2"/>
+      <geom type="sphere" size="0.035" rgba="0 0 1 0.8" mass="0.2"/>
       <site name="payload_connection_site_2" pos="0.0 0.0 0.0"/>
     </body>

File: model/scene_acro_payload_lidar.xml.xacro (robot description, xacro)
@@ -76,5 +76,5 @@
       <joint name="payload_y" type="slide" axis="0 1 0" damping="0.2"/>
       <joint name="payload_z" type="slide" axis="0 0 1" damping="0.2"/>
-      <geom type="sphere" size="0.03" rgba="0 0 1 0.8" mass="0.2"/>
+      <geom type="sphere" size="0.035" rgba="0 0 1 0.8" mass="0.2"/>
       <site name="payload_connection_site" pos="0.0 0.0 0.0"/>
     </body>
@@ -83,5 +83,5 @@
       <joint name="payload_2_y" type="slide" axis="0 1 0" damping="0.2"/>
       <joint name="payload_2_z" type="slide" axis="0 0 1" damping="0.2"/>
-      <geom type="sphere" size="0.03" rgba="0 0 1 0.8" mass="0.2"/>
+      <geom type="sphere" size="0.035" rgba="0 0 1 0.8" mass="0.2"/>
       <site name="payload_connection_site_2" pos="0.0 0.0 0.0"/>
     </body>

File: model/scene_inertial_force_sphere.xml.xacro (robot description, xacro)
@@ -13,5 +13,5 @@
   <xacro:arg name="payload_y" default="0.0"/>
   <xacro:arg name="payload_z" default="0.29"/>
-  <xacro:arg name="payload_radius" default="0.03"/>
+  <xacro:arg name="payload_radius" default="0.035"/>
   <xacro:arg name="payload_mass" default="0.2"/>
   <xacro:arg name="payload_damping" default="0.2"/>

File: model/scene_lowlevel.xml.xacro (robot description, xacro)
@@ -40,6 +40,6 @@
       <joint name="payload_y" type="slide" axis="0 1 0" damping="0.2"/>
       <joint name="payload_z" type="slide" axis="0 0 1" damping="0.2"/>
-      <geom type="sphere" size="0.03" rgba="0 0 1 0.8" mass="0.1128"/>
-      <site name="payload_connection_site" pos="0.0 0.0 0.03"/>
+      <geom type="sphere" size="0.035" rgba="0 0 1 0.8" mass="0.1128"/>
+      <site name="payload_connection_site" pos="0.0 0.0 0.035"/>
     </body>
     <geom name="origin_x" type="cylinder" fromto="0 0 0.01 0.5 0 0.01" size="0.01" rgba="1 0 0 0.1" contype="0" conaffinity="0" group="1"/>

File: model/scene_so3.xml.xacro (robot description, xacro)
@@ -41,6 +41,6 @@
       <joint name="payload_y" type="slide" axis="0 1 0" damping="0.2"/>
       <joint name="payload_z" type="slide" axis="0 0 1" damping="0.2"/>
-      <geom type="sphere" size="0.03" rgba="0 0 1 0.8" mass="0.1128"/>
-      <site name="payload_connection_site" pos="0.0 0.0 0.03"/>
+      <geom type="sphere" size="0.035" rgba="0 0 1 0.8" mass="0.1128"/>
+      <site name="payload_connection_site" pos="0.0 0.0 0.035"/>
     </body>
     <geom name="wall_back" type="box" pos="-3 0 1.5" size="0.05 2 1.5" rgba="0.8 0.8 0.8 0.2"/>

Commit message: Expose IMU and acro sensor noise parameters

File: model/quadrotor_acro_macro.xml.xacro (robot description, xacro)
@@ -271,8 +271,11 @@
   </xacro:macro>
   <xacro:macro name="quadrotor_physical_sensors" params="prefix">
-    <accelerometer name="${prefix}_accel" site="${prefix}_imu" />
-    <gyro name="${prefix}_gyro" site="${prefix}_imu" />
-  </xacro:macro>
-  <xacro:macro name="quadrotor_actuators" params="prefix control_hz:=240">
+    <!-- Keep MuJoCo's native sensor noise at zero. Measurement noise is added
+         only by ImuPublisher so that one model controls it unambiguously. -->
+    <accelerometer name="${prefix}_accel" site="${prefix}_imu" noise="0.0" />
+    <gyro name="${prefix}_gyro" site="${prefix}_imu" noise="0.0" />
+  </xacro:macro>
+  <xacro:macro name="quadrotor_actuators"
+               params="prefix control_hz:=240 acro_gyro_noise_density:=2.5e-3 acro_gyro_bias_rw:=0.0">
     <plugin site="${prefix}_rotor1_site" name="${prefix}_rotor1"
             plugin="MujocoRosUtils::RotorMotor"
@@ -325,7 +328,14 @@
       <config key="control_hz"   value="${control_hz}"/>
       <config key="body_name"    value="${prefix}"/>
-    </plugin>
-  </xacro:macro>
-  <xacro:macro name="quadrotor_sensor_plugins" params="prefix odom_hz:=240 imu_hz:=350">
+      <config key="gyro_noise_density" value="${acro_gyro_noise_density}"/>
+      <config key="gyro_bias_rw" value="${acro_gyro_bias_rw}"/>
+      <config key="gyro_bias_init_x" value="0.0"/>
+      <config key="gyro_bias_init_y" value="0.0"/>
+      <config key="gyro_bias_init_z" value="0.0"/>
+      <config key="gyro_range" value="0.0"/>
+    </plugin>
+  </xacro:macro>
+  <xacro:macro name="quadrotor_sensor_plugins"
+               params="prefix odom_hz:=240 imu_hz:=350 imu_gyro_noise_density:=2.5e-3 imu_accel_noise_density:=1.8e-3 imu_gyro_bias_rw:=0.0 imu_accel_bias_rw:=0.0">
     <plugin name="${prefix}_odom" plugin="MujocoRosUtils::OdometryPublisher" objtype="xbody" objname="${prefix}">
       <config key="publish_rate" value="${odom_hz}"/>
@@ -336,4 +346,16 @@
       <config key="gyro_sensor"  value="${prefix}_gyro"/>
       <config key="publish_rate" value="${imu_hz}"/>
+      <config key="gyro_noise_density" value="${imu_gyro_noise_density}"/>
+      <config key="gyro_bias_rw" value="${imu_gyro_bias_rw}"/>
+      <config key="gyro_bias_init_x" value="0.0"/>
+      <config key="gyro_bias_init_y" value="0.0"/>
+      <config key="gyro_bias_init_z" value="0.0"/>
+      <config key="gyro_range" value="0.0"/>
+      <config key="accel_noise_density" value="${imu_accel_noise_density}"/>
+      <config key="accel_bias_rw" value="${imu_accel_bias_rw}"/>
+      <config key="accel_bias_init_x" value="0.0"/>
+      <config key="accel_bias_init_y" value="0.0"/>
+      <config key="accel_bias_init_z" value="0.0"/>
+      <config key="accel_range" value="0.0"/>
     </plugin>
   </xacro:macro>

File: model/scene_acro.xml.xacro (robot description, xacro)
@@ -20,4 +20,11 @@
   <xacro:arg name="clock_hz" default="400"/>
   <xacro:arg name="lidar_hz" default="10"/>
+  <!-- Sensor and rate-loop noise is applied by MujocoRosUtils. -->
+  <xacro:arg name="imu_gyro_noise_density" default="2.5e-3"/>
+  <xacro:arg name="imu_accel_noise_density" default="1.8e-3"/>
+  <xacro:arg name="imu_gyro_bias_rw" default="0.0"/>
+  <xacro:arg name="imu_accel_bias_rw" default="0.0"/>
+  <xacro:arg name="acro_gyro_noise_density" default="2.5e-3"/>
+  <xacro:arg name="acro_gyro_bias_rw" default="0.0"/>
   <xacro:include filename="quadrotor_acro_macro.xml.xacro" />
   <compiler angle="radian" meshdir="$(arg meshdir)"/>
@@ -83,5 +90,9 @@
   </worldbody>
   <actuator>
-    <xacro:quadrotor_actuators prefix="$(arg quad_name)" control_hz="$(arg control_hz)" />
+    <xacro:quadrotor_actuators
+        prefix="$(arg quad_name)"
+        control_hz="$(arg control_hz)"
+        acro_gyro_noise_density="$(arg acro_gyro_noise_density)"
+        acro_gyro_bias_rw="$(arg acro_gyro_bias_rw)" />
   </actuator>
   <tendon>
@@ -93,5 +104,12 @@
   <sensor>
     <xacro:quadrotor_physical_sensors prefix="$(arg quad_name)" />
-    <xacro:quadrotor_sensor_plugins prefix="$(arg quad_name)" odom_hz="$(arg odom_hz)" imu_hz="$(arg imu_hz)" />
+    <xacro:quadrotor_sensor_plugins
+        prefix="$(arg quad_name)"
+        odom_hz="$(arg odom_hz)"
+        imu_hz="$(arg imu_hz)"
+        imu_gyro_noise_density="$(arg imu_gyro_noise_density)"
+        imu_accel_noise_density="$(arg imu_accel_noise_density)"
+        imu_gyro_bias_rw="$(arg imu_gyro_bias_rw)"
+        imu_accel_bias_rw="$(arg imu_accel_bias_rw)" />
     <plugin name="payload_odom" plugin="MujocoRosUtils::OdometryPublisher" objtype="xbody" objname="payload">
       <config key="publish_rate" value="$(arg payload_odom_hz)"/>

File: model/scene_acro_gate.xml.xacro (robot description, xacro)
@@ -20,4 +20,10 @@
   <xacro:arg name="clock_hz" default="400"/>
   <xacro:arg name="lidar_hz" default="10"/>
+  <xacro:arg name="imu_gyro_noise_density" default="2.5e-3"/>
+  <xacro:arg name="imu_accel_noise_density" default="1.8e-3"/>
+  <xacro:arg name="imu_gyro_bias_rw" default="0.0"/>
+  <xacro:arg name="imu_accel_bias_rw" default="0.0"/>
+  <xacro:arg name="acro_gyro_noise_density" default="2.5e-3"/>
+  <xacro:arg name="acro_gyro_bias_rw" default="0.0"/>
   <xacro:arg name="gates_collide" default="0"/>
   <xacro:arg name="gate_radius" default="0.42"/>
@@ -112,5 +118,9 @@
   </worldbody>
   <actuator>
-    <xacro:quadrotor_actuators prefix="$(arg quad_name)" control_hz="$(arg control_hz)" />
+    <xacro:quadrotor_actuators
+        prefix="$(arg quad_name)"
+        control_hz="$(arg control_hz)"
+        acro_gyro_noise_density="$(arg acro_gyro_noise_density)"
+        acro_gyro_bias_rw="$(arg acro_gyro_bias_rw)" />
   </actuator>
   <tendon>
@@ -122,5 +132,12 @@
   <sensor>
     <xacro:quadrotor_physical_sensors prefix="$(arg quad_name)" />
-    <xacro:quadrotor_sensor_plugins prefix="$(arg quad_name)" odom_hz="$(arg odom_hz)" imu_hz="$(arg imu_hz)" />
+    <xacro:quadrotor_sensor_plugins
+        prefix="$(arg quad_name)"
+        odom_hz="$(arg odom_hz)"
+        imu_hz="$(arg imu_hz)"
+        imu_gyro_noise_density="$(arg imu_gyro_noise_density)"
+        imu_accel_noise_density="$(arg imu_accel_noise_density)"
+        imu_gyro_bias_rw="$(arg imu_gyro_bias_rw)"
+        imu_accel_bias_rw="$(arg imu_accel_bias_rw)" />
     <plugin name="payload_odom" plugin="MujocoRosUtils::OdometryPublisher" objtype="xbody" objname="payload">
       <config key="publish_rate" value="$(arg payload_odom_hz)"/>

File: model/scene_acro_lidar.xml.xacro (robot description, xacro)
@@ -20,4 +20,10 @@
   <xacro:arg name="clock_hz" default="400"/>
   <xacro:arg name="lidar_hz" default="10"/>
+  <xacro:arg name="imu_gyro_noise_density" default="2.5e-3"/>
+  <xacro:arg name="imu_accel_noise_density" default="1.8e-3"/>
+  <xacro:arg name="imu_gyro_bias_rw" default="0.0"/>
+  <xacro:arg name="imu_accel_bias_rw" default="0.0"/>
+  <xacro:arg name="acro_gyro_noise_density" default="2.5e-3"/>
+  <xacro:arg name="acro_gyro_bias_rw" default="0.0"/>
   <xacro:include filename="quadrotor_acro_macro.xml.xacro" />
   <compiler angle="radian" meshdir="$(arg meshdir)"/>
@@ -95,5 +101,9 @@
   </worldbody>
   <actuator>
-    <xacro:quadrotor_actuators prefix="$(arg quad_name)" control_hz="$(arg control_hz)" />
+    <xacro:quadrotor_actuators
+        prefix="$(arg quad_name)"
+        control_hz="$(arg control_hz)"
+        acro_gyro_noise_density="$(arg acro_gyro_noise_density)"
+        acro_gyro_bias_rw="$(arg acro_gyro_bias_rw)" />
   </actuator>
   <tendon>
@@ -105,5 +115,12 @@
   <sensor>
     <xacro:quadrotor_physical_sensors prefix="$(arg quad_name)" />
-    <xacro:quadrotor_sensor_plugins prefix="$(arg quad_name)" odom_hz="$(arg odom_hz)" imu_hz="$(arg imu_hz)" />
+    <xacro:quadrotor_sensor_plugins
+        prefix="$(arg quad_name)"
+        odom_hz="$(arg odom_hz)"
+        imu_hz="$(arg imu_hz)"
+        imu_gyro_noise_density="$(arg imu_gyro_noise_density)"
+        imu_accel_noise_density="$(arg imu_accel_noise_density)"
+        imu_gyro_bias_rw="$(arg imu_gyro_bias_rw)"
+        imu_accel_bias_rw="$(arg imu_accel_bias_rw)" />
     <xacro:quadrotor_lidar_plugin prefix="$(arg quad_name)" lidar_hz="$(arg lidar_hz)" />
     <plugin name="payload_odom" plugin="MujocoRosUtils::OdometryPublisher" objtype="xbody" objname="payload">

File: model/scene_acro_payload.xml.xacro (robot description, xacro)
@@ -20,4 +20,10 @@
   <xacro:arg name="clock_hz" default="400"/>
   <xacro:arg name="lidar_hz" default="10"/>
+  <xacro:arg name="imu_gyro_noise_density" default="2.5e-3"/>
+  <xacro:arg name="imu_accel_noise_density" default="1.8e-3"/>
+  <xacro:arg name="imu_gyro_bias_rw" default="0.0"/>
+  <xacro:arg name="imu_accel_bias_rw" default="0.0"/>
+  <xacro:arg name="acro_gyro_noise_density" default="2.5e-3"/>
+  <xacro:arg name="acro_gyro_bias_rw" default="0.0"/>
   <xacro:include filename="quadrotor_acro_macro.xml.xacro" />
   <compiler angle="radian" meshdir="$(arg meshdir)"/>
@@ -83,5 +89,9 @@
   </worldbody>
   <actuator>
-    <xacro:quadrotor_actuators prefix="$(arg quad_name)" control_hz="$(arg control_hz)" />
+    <xacro:quadrotor_actuators
+        prefix="$(arg quad_name)"
+        control_hz="$(arg control_hz)"
+        acro_gyro_noise_density="$(arg acro_gyro_noise_density)"
+        acro_gyro_bias_rw="$(arg acro_gyro_bias_rw)" />
   </actuator>
   <tendon>
@@ -93,5 +103,12 @@
   <sensor>
     <xacro:quadrotor_physical_sensors prefix="$(arg quad_name)" />
-    <xacro:quadrotor_sensor_plugins prefix="$(arg quad_name)" odom_hz="$(arg odom_hz)" imu_hz="$(arg imu_hz)" />
+    <xacro:quadrotor_sensor_plugins
+        prefix="$(arg quad_name)"
+        odom_hz="$(arg odom_hz)"
+        imu_hz="$(arg imu_hz)"
+        imu_gyro_noise_density="$(arg imu_gyro_noise_density)"
+        imu_accel_noise_density="$(arg imu_accel_noise_density)"
+        imu_gyro_bias_rw="$(arg imu_gyro_bias_rw)"
+        imu_accel_bias_rw="$(arg imu_accel_bias_rw)" />
     <plugin name="payload_odom" plugin="MujocoRosUtils::OdometryPublisher" objtype="xbody" objname="payload">
       <config key="publish_rate" value="$(arg payload_odom_hz)"/>

File: model/scene_acro_payload_lidar.xml.xacro (robot description, xacro)
@@ -20,4 +20,10 @@
   <xacro:arg name="clock_hz" default="400"/>
   <xacro:arg name="lidar_hz" default="10"/>
+  <xacro:arg name="imu_gyro_noise_density" default="2.5e-3"/>
+  <xacro:arg name="imu_accel_noise_density" default="1.8e-3"/>
+  <xacro:arg name="imu_gyro_bias_rw" default="0.0"/>
+  <xacro:arg name="imu_accel_bias_rw" default="0.0"/>
+  <xacro:arg name="acro_gyro_noise_density" default="2.5e-3"/>
+  <xacro:arg name="acro_gyro_bias_rw" default="0.0"/>
   <xacro:include filename="quadrotor_acro_macro.xml.xacro" />
   <compiler angle="radian" meshdir="$(arg meshdir)"/>
@@ -95,5 +101,9 @@
   </worldbody>
   <actuator>
-    <xacro:quadrotor_actuators prefix="$(arg quad_name)" control_hz="$(arg control_hz)" />
+    <xacro:quadrotor_actuators
+        prefix="$(arg quad_name)"
+        control_hz="$(arg control_hz)"
+        acro_gyro_noise_density="$(arg acro_gyro_noise_density)"
+        acro_gyro_bias_rw="$(arg acro_gyro_bias_rw)" />
   </actuator>
   <tendon>
@@ -105,5 +115,12 @@
   <sensor>
     <xacro:quadrotor_physical_sensors prefix="$(arg quad_name)" />
-    <xacro:quadrotor_sensor_plugins prefix="$(arg quad_name)" odom_hz="$(arg odom_hz)" imu_hz="$(arg imu_hz)" />
+    <xacro:quadrotor_sensor_plugins
+        prefix="$(arg quad_name)"
+        odom_hz="$(arg odom_hz)"
+        imu_hz="$(arg imu_hz)"
+        imu_gyro_noise_density="$(arg imu_gyro_noise_density)"
+        imu_accel_noise_density="$(arg imu_accel_noise_density)"
+        imu_gyro_bias_rw="$(arg imu_gyro_bias_rw)"
+        imu_accel_bias_rw="$(arg imu_accel_bias_rw)" />
     <xacro:quadrotor_lidar_plugin prefix="$(arg quad_name)" lidar_hz="$(arg lidar_hz)" />
     <plugin name="payload_odom" plugin="MujocoRosUtils::OdometryPublisher" objtype="xbody" objname="payload">

Commit message: Align payload damping and add onboard camera

File: model/quadrotor_acro_macro.xml.xacro (robot description, xacro)
@@ -173,4 +173,8 @@
             density="0" contype="0" conaffinity="0" group="2"/>
       <site name="${prefix}_imu" pos="0 0 0" size="0.001" rgba="0 0 0 0" group="5"/>
+       <camera name="${prefix}_camera"
+            pos="0.03 0 -0.04"
+            xyaxes="0 -1 0 1 0 0"
+            fovy="75"/>
       <xacro:if value="${include_lidar}">
         <!--

File: model/scene_acro_payload.xml.xacro (robot description, xacro)
@@ -67,14 +67,14 @@
                           primitive_alpha="$(arg primitive_alpha)" />
     <body name="payload" pos="-0.7 0.0 0.02">
-      <joint name="payload_x" type="slide" axis="1 0 0" damping="0.2"/>
-      <joint name="payload_y" type="slide" axis="0 1 0" damping="0.2"/>
-      <joint name="payload_z" type="slide" axis="0 0 1" damping="0.2"/>
+      <joint name="payload_x" type="slide" axis="1 0 0" damping="0.06"/>
+      <joint name="payload_y" type="slide" axis="0 1 0" damping="0.06"/>
+      <joint name="payload_z" type="slide" axis="0 0 1" damping="0.06"/>
       <geom type="sphere" size="0.035" rgba="0 0 1 0.8" mass="0.2"/>
       <site name="payload_connection_site" pos="0.0 0.0 0.0"/>
     </body>
     <body name="payload_2" pos="-0.7 0.7 0.02">
-      <joint name="payload_2_x" type="slide" axis="1 0 0" damping="0.2"/>
-      <joint name="payload_2_y" type="slide" axis="0 1 0" damping="0.2"/>
-      <joint name="payload_2_z" type="slide" axis="0 0 1" damping="0.2"/>
+      <joint name="payload_2_x" type="slide" axis="1 0 0" damping="0.06"/>
+      <joint name="payload_2_y" type="slide" axis="0 1 0" damping="0.06"/>
+      <joint name="payload_2_z" type="slide" axis="0 0 1" damping="0.06"/>
       <geom type="sphere" size="0.035" rgba="0 0 1 0.8" mass="0.2"/>
       <site name="payload_connection_site_2" pos="0.0 0.0 0.0"/>

File: model/scene_acro_payload_lidar.xml.xacro (robot description, xacro)
@@ -79,14 +79,14 @@
                           include_lidar="true" />
     <body name="payload" pos="-0.7 0.0 0.02">
-      <joint name="payload_x" type="slide" axis="1 0 0" damping="0.2"/>
-      <joint name="payload_y" type="slide" axis="0 1 0" damping="0.2"/>
-      <joint name="payload_z" type="slide" axis="0 0 1" damping="0.2"/>
+      <joint name="payload_x" type="slide" axis="1 0 0" damping="0.06"/>
+      <joint name="payload_y" type="slide" axis="0 1 0" damping="0.06"/>
+      <joint name="payload_z" type="slide" axis="0 0 1" damping="0.06"/>
       <geom type="sphere" size="0.035" rgba="0 0 1 0.8" mass="0.2"/>
       <site name="payload_connection_site" pos="0.0 0.0 0.0"/>
     </body>
     <body name="payload_2" pos="-0.7 0.7 0.02">
-      <joint name="payload_2_x" type="slide" axis="1 0 0" damping="0.2"/>
-      <joint name="payload_2_y" type="slide" axis="0 1 0" damping="0.2"/>
-      <joint name="payload_2_z" type="slide" axis="0 0 1" damping="0.2"/>
+      <joint name="payload_2_x" type="slide" axis="1 0 0" damping="0.06"/>
+      <joint name="payload_2_y" type="slide" axis="0 1 0" damping="0.06"/>
+      <joint name="payload_2_z" type="slide" axis="0 0 1" damping="0.06"/>
       <geom type="sphere" size="0.035" rgba="0 0 1 0.8" mass="0.2"/>
       <site name="payload_connection_site_2" pos="0.0 0.0 0.0"/>
