Commit message: Parameterize payload plant and headless duration

File: model/quadrotor_acro_macro.xml.xacro (robot description, xacro)
@@ -4,14 +4,15 @@
     <!-- The quadrotor is intentionally primitive-only; no external mesh asset is required. -->
   </xacro:macro>
-  <xacro:macro name="quadrotor_body" params="prefix pos euler:='0 0 0' mesh_pos:='-0.17 -0.16 -0.1' mesh_euler:='0 1.57 1.57079632679' primitive_alpha:='1.0' include_lidar:='false'">
+  <xacro:macro name="quadrotor_body" params="prefix pos euler:='0 0 0' mesh_pos:='-0.17 -0.16 -0.1' mesh_euler:='0 1.57 1.57079632679' primitive_alpha:='1.0' include_lidar:='false'
+                      mass:=1.24 ixx:=0.0027338143976 iyy:=0.0027336327812 izz:=0.0052991944907">
     <body name="${prefix}" pos="${pos}" euler="${euler}">
       <joint name="${prefix}" type="free" damping="0.001" armature="0" pos="0 0 0"/>
       <!--
-        Preserve the original 1.24 kg rigid-body dynamics exactly. The
+        Defaults preserve the original 1.24 kg rigid-body dynamics. The
         physical geoms below retain the previous collision and fluid-drag
         envelopes, but no longer contribute mass because inertia is explicit.
       -->
-      <inertial pos="0 0 0.0004838709677" mass="1.24"
-                diaginertia="0.0027338143976 0.0027336327812 0.0052991944907"/>
+      <inertial pos="0 0 0.0004838709677" mass="${mass}"
+                diaginertia="${ixx} ${iyy} ${izz}"/>
       <!-- Hidden physical proxies: keep group 0 so other simulated LiDARs see the vehicle. -->
       <geom name="${prefix}_core" type="box" size="0.035 0.035 0.015"
@@ -173,8 +174,8 @@
             density="0" contype="0" conaffinity="0" group="2"/>
       <site name="${prefix}_imu" pos="0 0 0" size="0.001" rgba="0 0 0 0" group="5"/>
-      <!--<camera name="${prefix}_camera"
+      <camera name="${prefix}_camera"
             pos="0.03 0 -0.04"
             xyaxes="0 -1 0 1 0 0"
-            fovy="75"/> -->
+            fovy="75"/>
       <xacro:if value="${include_lidar}">
         <!--

File: model/scene_acro_payload.xml.xacro (robot description, xacro)
@@ -8,4 +8,13 @@
   <xacro:arg name="init_pitch" default="0.0"/>
   <xacro:arg name="init_yaw"   default="0.0"/>
+  <xacro:arg name="payload_x" default="-0.7"/>
+  <xacro:arg name="payload_y" default="0.0"/>
+  <xacro:arg name="payload_z" default="0.02"/>
+  <xacro:arg name="quadrotor_mass" default="1.24"/>
+  <xacro:arg name="quadrotor_ixx" default="0.0027338143976"/>
+  <xacro:arg name="quadrotor_iyy" default="0.0027336327812"/>
+  <xacro:arg name="quadrotor_izz" default="0.0052991944907"/>
+  <xacro:arg name="payload_mass" default="0.2"/>
+  <xacro:arg name="cable_length" default="0.95"/>
   <xacro:arg name="meshdir" default="."/>
   <xacro:arg name="mesh_pos" default="-0.17 -0.16 -0.1"/>
@@ -63,12 +72,16 @@
                           pos="$(arg init_x) $(arg init_y) $(arg init_z)"
                           euler="$(arg init_roll) $(arg init_pitch) $(arg init_yaw)"
+                          mass="$(arg quadrotor_mass)"
+                          ixx="$(arg quadrotor_ixx)"
+                          iyy="$(arg quadrotor_iyy)"
+                          izz="$(arg quadrotor_izz)"
                           mesh_pos="$(arg mesh_pos)"
                           mesh_euler="$(arg mesh_euler)"
                           primitive_alpha="$(arg primitive_alpha)" />
-    <body name="payload" pos="-0.7 0.0 0.02">
+    <body name="payload" pos="$(arg payload_x) $(arg payload_y) $(arg payload_z)">
       <joint name="payload_x" type="slide" axis="1 0 0" damping="0.06"/>
       <joint name="payload_y" type="slide" axis="0 1 0" damping="0.06"/>
       <joint name="payload_z" type="slide" axis="0 0 1" damping="0.06"/>
-      <geom type="sphere" size="0.035" rgba="0 0 1 0.8" mass="0.2"/>
+      <geom type="sphere" size="0.035" rgba="0 0 1 0.8" mass="$(arg payload_mass)"/>
       <site name="payload_connection_site" pos="0.0 0.0 0.0"/>
     </body>
@@ -96,5 +109,5 @@
   </actuator>
   <tendon>
-    <spatial name="rope0" limited="true" range="0 0.95" width=".0005">
+    <spatial name="rope0" limited="true" range="0 $(arg cable_length)" width=".0005">
       <site site="$(arg quad_name)_payload_site"/>
       <site site="payload_connection_site"/>

Commit message: px4 interface

File: model/quadrotor_acro_macro.xml.xacro (robot description, xacro)
@@ -282,6 +282,6 @@
     <gyro name="${prefix}_gyro" site="${prefix}_imu" noise="0.0" />
   </xacro:macro>
-  <xacro:macro name="quadrotor_actuators"
-               params="prefix control_hz:=240 acro_gyro_noise_density:=2.5e-3 acro_gyro_bias_rw:=0.0">
+  <!-- The plant can also be driven by an external flight controller. -->
+  <xacro:macro name="quadrotor_rotor_actuators" params="prefix delay_samples:=8">
     <plugin site="${prefix}_rotor1_site" name="${prefix}_rotor1"
             plugin="MujocoRosUtils::RotorMotor"
@@ -289,5 +289,5 @@
             ctrlrange="0 3000.0"
             gear="0 0 1 0 0 0.015"
-            nsample="8" delay="0.018" interp="zoh">
+            nsample="${delay_samples}" delay="0.018" interp="zoh">
       <config key="kf" value="2.063751543951938e-06"/>
       <config key="tau" value="0.025"/>
@@ -298,5 +298,5 @@
             ctrlrange="0 3000.0"
             gear="0 0 1 0 0 -0.015"
-            nsample="8" delay="0.018" interp="zoh">
+            nsample="${delay_samples}" delay="0.018" interp="zoh">
       <config key="kf" value="2.063751543951938e-06"/>
       <config key="tau" value="0.025"/>
@@ -307,5 +307,5 @@
             ctrlrange="0 3000.0"
             gear="0 0 1 0 0 -0.015"
-            nsample="8" delay="0.018" interp="zoh">
+            nsample="${delay_samples}" delay="0.018" interp="zoh">
       <config key="kf" value="2.063751543951938e-06"/>
       <config key="tau" value="0.025"/>
@@ -316,8 +316,13 @@
             ctrlrange="0 3000.0"
             gear="0 0 1 0 0 0.015"
-            nsample="8" delay="0.018" interp="zoh">
+            nsample="${delay_samples}" delay="0.018" interp="zoh">
       <config key="kf" value="2.063751543951938e-06"/>
       <config key="tau" value="0.025"/>
     </plugin>
+  </xacro:macro>
+  <xacro:macro name="quadrotor_actuators"
+               params="prefix control_hz:=240 acro_gyro_noise_density:=2.5e-3 acro_gyro_bias_rw:=0.0 controller_backend:=acro">
+    <xacro:quadrotor_rotor_actuators prefix="${prefix}" delay_samples="${32 if controller_backend == 'px4' else 8}"/>
+    <xacro:unless value="${controller_backend == 'px4'}">
     <plugin name="acro_ctrl_${prefix}" plugin="MujocoRosUtils::AcroMode" joint="${prefix}">
       <config key="actuator_r1"  value="${prefix}_rotor1"/>
@@ -340,4 +345,12 @@
       <config key="gyro_bias_init_z" value="0.0"/>
       <config key="gyro_range" value="0.0"/>
+    </plugin>
+    </xacro:unless>
+  </xacro:macro>
+  <xacro:macro name="quadrotor_mavlink" params="prefix simulator_port:=4560 csv_path:=''">
+    <plugin name="${prefix}_mavlink" plugin="MujocoRosUtils::MavlinkInterface">
+      <config key="body_name" value="${prefix}"/>
+      <config key="simulator_port" value="${simulator_port}"/>
+      <config key="csv_path" value="${csv_path}"/>
     </plugin>
   </xacro:macro>
