Commit message: Increase simulated payload damping to 0.2

File: model/scene.xml.xacro (robot description, xacro)
@@ -39,7 +39,7 @@
     <xacro:quadrotor_body prefix="$(arg quad_name)" pos="$(arg init_x) $(arg init_y) $(arg init_z)" euler="$(arg init_roll) $(arg init_pitch) $(arg init_yaw)" />
     <body name="payload" pos="1 0 0.02">
-      <joint name="payload_x" type="slide" axis="1 0 0" damping="0.1"/>
-      <joint name="payload_y" type="slide" axis="0 1 0" damping="0.1"/>
-      <joint name="payload_z" type="slide" axis="0 0 1" damping="0.1"/>
+      <joint name="payload_x" type="slide" axis="1 0 0" damping="0.2"/>
+      <joint name="payload_y" type="slide" axis="0 1 0" damping="0.2"/>
+      <joint name="payload_z" type="slide" axis="0 0 1" damping="0.2"/>
       <geom type="sphere" size="0.03" rgba="0 0 1 0.8" mass="0.1"/>
       <site name="payload_connection_site" pos="0.0 0.0 0.03"/>

File: model/scene_acro.xml.xacro (robot description, xacro)
@@ -61,14 +61,14 @@
                           primitive_alpha="$(arg primitive_alpha)" />
     <body name="payload" pos="-0.7 0.0 0.02">
-      <joint name="payload_x" type="slide" axis="1 0 0" damping="0.1"/>
-      <joint name="payload_y" type="slide" axis="0 1 0" damping="0.1"/>
-      <joint name="payload_z" type="slide" axis="0 0 1" damping="0.1"/>
+      <joint name="payload_x" type="slide" axis="1 0 0" damping="0.2"/>
+      <joint name="payload_y" type="slide" axis="0 1 0" damping="0.2"/>
+      <joint name="payload_z" type="slide" axis="0 0 1" damping="0.2"/>
       <geom type="sphere" size="0.03" rgba="0 0 1 0.8" mass="0.2"/>
       <site name="payload_connection_site" pos="0.0 0.0 0.0"/>
     </body>
     <body name="payload_2" pos="-0.7 0.7 0.02">
-      <joint name="payload_2_x" type="slide" axis="1 0 0" damping="0.1"/>
-      <joint name="payload_2_y" type="slide" axis="0 1 0" damping="0.1"/>
-      <joint name="payload_2_z" type="slide" axis="0 0 1" damping="0.1"/>
+      <joint name="payload_2_x" type="slide" axis="1 0 0" damping="0.2"/>
+      <joint name="payload_2_y" type="slide" axis="0 1 0" damping="0.2"/>
+      <joint name="payload_2_z" type="slide" axis="0 0 1" damping="0.2"/>
       <geom type="sphere" size="0.03" rgba="0 0 1 0.8" mass="0.2"/>
       <site name="payload_connection_site_2" pos="0.0 0.0 0.0"/>

File: model/scene_acro_gate.xml.xacro (robot description, xacro)
@@ -86,14 +86,14 @@
                           primitive_alpha="$(arg primitive_alpha)" />
     <body name="payload" pos="-0.0 0.0 0.7">
-      <joint name="payload_x" type="slide" axis="1 0 0" damping="0.1"/>
-      <joint name="payload_y" type="slide" axis="0 1 0" damping="0.1"/>
-      <joint name="payload_z" type="slide" axis="0 0 1" damping="0.1"/>
+      <joint name="payload_x" type="slide" axis="1 0 0" damping="0.2"/>
+      <joint name="payload_y" type="slide" axis="0 1 0" damping="0.2"/>
+      <joint name="payload_z" type="slide" axis="0 0 1" damping="0.2"/>
       <geom type="sphere" size="0.03" rgba="0 0 1 0.8" mass="0.2"/>
       <site name="payload_connection_site" pos="0.0 0.0 0.0"/>
     </body>
     <body name="payload_2" pos="-0.7 0.7 0.02">
-      <joint name="payload_2_x" type="slide" axis="1 0 0" damping="0.1"/>
-      <joint name="payload_2_y" type="slide" axis="0 1 0" damping="0.1"/>
-      <joint name="payload_2_z" type="slide" axis="0 0 1" damping="0.1"/>
+      <joint name="payload_2_x" type="slide" axis="1 0 0" damping="0.2"/>
+      <joint name="payload_2_y" type="slide" axis="0 1 0" damping="0.2"/>
+      <joint name="payload_2_z" type="slide" axis="0 0 1" damping="0.2"/>
       <geom type="sphere" size="0.03" rgba="0 0 1 0.8" mass="0.2"/>
       <site name="payload_connection_site_2" pos="0.0 0.0 0.0"/>

File: model/scene_acro_humanoid.xml.xacro (robot description, xacro)
@@ -39,7 +39,7 @@
     <xacro:g1_humanoid_body prefix="g1" pos="3 0 0.793" euler="0 0 0"/>
     <body name="payload" pos="0.8 0 0.02">
-      <joint name="payload_x" type="slide" axis="1 0 0" damping="0.1"/>
-      <joint name="payload_y" type="slide" axis="0 1 0" damping="0.1"/>
-      <joint name="payload_z" type="slide" axis="0 0 1" damping="0.1"/>
+      <joint name="payload_x" type="slide" axis="1 0 0" damping="0.2"/>
+      <joint name="payload_y" type="slide" axis="0 1 0" damping="0.2"/>
+      <joint name="payload_z" type="slide" axis="0 0 1" damping="0.2"/>
       <geom type="sphere" size="0.03" rgba="0 0 1 0.8" mass="0.1128"/>
       <site name="payload_connection_site" pos="0.0 0.0 0.03"/>

File: model/scene_acro_lidar.xml.xacro (robot description, xacro)
@@ -73,14 +73,14 @@
                           include_lidar="true" />
     <body name="payload" pos="-0.7 0.0 0.02">
-      <joint name="payload_x" type="slide" axis="1 0 0" damping="0.1"/>
-      <joint name="payload_y" type="slide" axis="0 1 0" damping="0.1"/>
-      <joint name="payload_z" type="slide" axis="0 0 1" damping="0.1"/>
+      <joint name="payload_x" type="slide" axis="1 0 0" damping="0.2"/>
+      <joint name="payload_y" type="slide" axis="0 1 0" damping="0.2"/>
+      <joint name="payload_z" type="slide" axis="0 0 1" damping="0.2"/>
       <geom type="sphere" size="0.03" rgba="0 0 1 0.8" mass="0.2"/>
       <site name="payload_connection_site" pos="0.0 0.0 0.0"/>
     </body>
     <body name="payload_2" pos="-0.7 0.7 0.02">
-      <joint name="payload_2_x" type="slide" axis="1 0 0" damping="0.1"/>
-      <joint name="payload_2_y" type="slide" axis="0 1 0" damping="0.1"/>
-      <joint name="payload_2_z" type="slide" axis="0 0 1" damping="0.1"/>
+      <joint name="payload_2_x" type="slide" axis="1 0 0" damping="0.2"/>
+      <joint name="payload_2_y" type="slide" axis="0 1 0" damping="0.2"/>
+      <joint name="payload_2_z" type="slide" axis="0 0 1" damping="0.2"/>
       <geom type="sphere" size="0.03" rgba="0 0 1 0.8" mass="0.2"/>
       <site name="payload_connection_site_2" pos="0.0 0.0 0.0"/>

File: model/scene_acro_multiple.xml.xacro (robot description, xacro)
@@ -46,7 +46,7 @@
     <xacro:quadrotor_body prefix="$(arg quad_name_2)" pos="$(arg init_x_2) $(arg init_y_2) $(arg init_z_2)" euler="$(arg init_roll_2) $(arg init_pitch_2) $(arg init_yaw_2)" />
     <body name="payload" pos="0.3 0.3 1.0">
-      <joint name="payload_x" type="slide" axis="1 0 0" damping="0.1"/>
-      <joint name="payload_y" type="slide" axis="0 1 0" damping="0.1"/>
-      <joint name="payload_z" type="slide" axis="0 0 1" damping="0.1"/>
+      <joint name="payload_x" type="slide" axis="1 0 0" damping="0.2"/>
+      <joint name="payload_y" type="slide" axis="0 1 0" damping="0.2"/>
+      <joint name="payload_z" type="slide" axis="0 0 1" damping="0.2"/>
       <geom type="sphere" size="0.03" rgba="0 0 1 0.8" mass="0.1128"/>
       <site name="payload_connection_site" pos="0.0 0.0 0.03"/>

File: model/scene_acro_payload.xml.xacro (robot description, xacro)
@@ -61,14 +61,14 @@
                           primitive_alpha="$(arg primitive_alpha)" />
     <body name="payload" pos="-0.7 0.0 0.02">
-      <joint name="payload_x" type="slide" axis="1 0 0" damping="0.1"/>
-      <joint name="payload_y" type="slide" axis="0 1 0" damping="0.1"/>
-      <joint name="payload_z" type="slide" axis="0 0 1" damping="0.1"/>
+      <joint name="payload_x" type="slide" axis="1 0 0" damping="0.2"/>
+      <joint name="payload_y" type="slide" axis="0 1 0" damping="0.2"/>
+      <joint name="payload_z" type="slide" axis="0 0 1" damping="0.2"/>
       <geom type="sphere" size="0.03" rgba="0 0 1 0.8" mass="0.2"/>
       <site name="payload_connection_site" pos="0.0 0.0 0.0"/>
     </body>
     <body name="payload_2" pos="-0.7 0.7 0.02">
-      <joint name="payload_2_x" type="slide" axis="1 0 0" damping="0.1"/>
-      <joint name="payload_2_y" type="slide" axis="0 1 0" damping="0.1"/>
-      <joint name="payload_2_z" type="slide" axis="0 0 1" damping="0.1"/>
+      <joint name="payload_2_x" type="slide" axis="1 0 0" damping="0.2"/>
+      <joint name="payload_2_y" type="slide" axis="0 1 0" damping="0.2"/>
+      <joint name="payload_2_z" type="slide" axis="0 0 1" damping="0.2"/>
       <geom type="sphere" size="0.03" rgba="0 0 1 0.8" mass="0.2"/>
       <site name="payload_connection_site_2" pos="0.0 0.0 0.0"/>

File: model/scene_acro_payload_lidar.xml.xacro (robot description, xacro)
@@ -73,14 +73,14 @@
                           include_lidar="true" />
     <body name="payload" pos="-0.7 0.0 0.02">
-      <joint name="payload_x" type="slide" axis="1 0 0" damping="0.1"/>
-      <joint name="payload_y" type="slide" axis="0 1 0" damping="0.1"/>
-      <joint name="payload_z" type="slide" axis="0 0 1" damping="0.1"/>
+      <joint name="payload_x" type="slide" axis="1 0 0" damping="0.2"/>
+      <joint name="payload_y" type="slide" axis="0 1 0" damping="0.2"/>
+      <joint name="payload_z" type="slide" axis="0 0 1" damping="0.2"/>
       <geom type="sphere" size="0.03" rgba="0 0 1 0.8" mass="0.2"/>
       <site name="payload_connection_site" pos="0.0 0.0 0.0"/>
     </body>
     <body name="payload_2" pos="-0.7 0.7 0.02">
-      <joint name="payload_2_x" type="slide" axis="1 0 0" damping="0.1"/>
-      <joint name="payload_2_y" type="slide" axis="0 1 0" damping="0.1"/>
-      <joint name="payload_2_z" type="slide" axis="0 0 1" damping="0.1"/>
+      <joint name="payload_2_x" type="slide" axis="1 0 0" damping="0.2"/>
+      <joint name="payload_2_y" type="slide" axis="0 1 0" damping="0.2"/>
+      <joint name="payload_2_z" type="slide" axis="0 0 1" damping="0.2"/>
       <geom type="sphere" size="0.03" rgba="0 0 1 0.8" mass="0.2"/>
       <site name="payload_connection_site_2" pos="0.0 0.0 0.0"/>

File: model/scene_inertial_force_sphere.xml.xacro (robot description, xacro)
@@ -15,5 +15,5 @@
   <xacro:arg name="payload_radius" default="0.03"/>
   <xacro:arg name="payload_mass" default="0.2"/>
-  <xacro:arg name="payload_damping" default="0.1"/>
+  <xacro:arg name="payload_damping" default="0.2"/>
   <xacro:arg name="cable_length" default="0.71"/>
   <xacro:arg name="publish_rate" default="240"/>

File: model/scene_lowlevel.xml.xacro (robot description, xacro)
@@ -37,7 +37,7 @@
     <xacro:quadrotor_body prefix="$(arg quad_name)" pos="$(arg init_x) $(arg init_y) $(arg init_z)" euler="$(arg init_roll) $(arg init_pitch) $(arg init_yaw)" />
     <body name="payload" pos="0.6 0 0.02">
-      <joint name="payload_x" type="slide" axis="1 0 0" damping="0.1"/>
-      <joint name="payload_y" type="slide" axis="0 1 0" damping="0.1"/>
-      <joint name="payload_z" type="slide" axis="0 0 1" damping="0.1"/>
+      <joint name="payload_x" type="slide" axis="1 0 0" damping="0.2"/>
+      <joint name="payload_y" type="slide" axis="0 1 0" damping="0.2"/>
+      <joint name="payload_z" type="slide" axis="0 0 1" damping="0.2"/>
       <geom type="sphere" size="0.03" rgba="0 0 1 0.8" mass="0.1128"/>
       <site name="payload_connection_site" pos="0.0 0.0 0.03"/>

File: model/scene_so3.xml.xacro (robot description, xacro)
@@ -38,7 +38,7 @@
     <xacro:quadrotor_body prefix="$(arg quad_name)" pos="$(arg init_x) $(arg init_y) $(arg init_z)" euler="$(arg init_roll) $(arg init_pitch) $(arg init_yaw)" />
     <body name="payload" pos="0.6 0 0.02">
-      <joint name="payload_x" type="slide" axis="1 0 0" damping="0.1"/>
-      <joint name="payload_y" type="slide" axis="0 1 0" damping="0.1"/>
-      <joint name="payload_z" type="slide" axis="0 0 1" damping="0.1"/>
+      <joint name="payload_x" type="slide" axis="1 0 0" damping="0.2"/>
+      <joint name="payload_y" type="slide" axis="0 1 0" damping="0.2"/>
+      <joint name="payload_z" type="slide" axis="0 0 1" damping="0.2"/>
       <geom type="sphere" size="0.03" rgba="0 0 1 0.8" mass="0.1128"/>
       <site name="payload_connection_site" pos="0.0 0.0 0.03"/>
