Commit message: Add configurable circular gate to payload simulation

File: model/scene_acro_payload.xml.xacro (robot description, xacro)
@@ -17,4 +17,11 @@
   <xacro:arg name="payload_mass" default="0.2"/>
   <xacro:arg name="cable_length" default="0.95"/>
+  <!-- Optional gate: clear opening radius and full depth along world x. -->
+  <xacro:arg name="enable_gate" default="false"/>
+  <xacro:arg name="gate_x" default="1.75"/>
+  <xacro:arg name="gate_y" default="0.0"/>
+  <xacro:arg name="gate_z" default="2.0"/>
+  <xacro:arg name="gate_radius" default="0.4"/>
+  <xacro:arg name="gate_thickness" default="0.1"/>
   <xacro:arg name="meshdir" default="."/>
   <xacro:arg name="mesh_pos" default="-0.17 -0.16 -0.1"/>
@@ -37,4 +44,5 @@
   <xacro:arg name="acro_gyro_bias_rw" default="0.0"/>
   <xacro:include filename="quadrotor_acro_macro.xml.xacro" />
+  <xacro:include filename="circular_gate_macro.xml.xacro" />
   <compiler angle="radian" meshdir="$(arg meshdir)"/>
   <option timestep="$(arg simulation_timestep)" gravity="0 0 -9.81" density="1.225" viscosity="1.8e-05" integrator="RK4" />
@@ -62,4 +70,5 @@
     <material name="mat_green" rgba="0.1 0.8 0.1 1" reflectance="0.01" shininess="0.01" specular="0.0" />
     <material name="mat_blue"  rgba="0.1 0.1 0.8 1" reflectance="0.01" shininess="0.01" specular="0.0" />
+    <material name="mat_gate" rgba="0.95 0.25 0.15 1" reflectance="0.05" shininess="0.05" specular="0.1"/>
     <xacro:quadrotor_visual_assets />
     <texture type="skybox" builtin="flat" rgb1="0 0 0" rgb2="0 0 0" width="512" height="3072"/>
@@ -78,4 +87,10 @@
     <geom class="environment" name="box_green" type="box" pos="4 -1 0.1" size="0.2 0.2 0.1" material="mat_green" />
     <geom class="environment" name="box_blue" type="box" pos="6 1 0.1" size="0.2 0.2 0.1" material="mat_blue" />
+    <xacro:if value="$(arg enable_gate)">
+      <xacro:circular_gate name="planner_gate"
+          pos="$(arg gate_x) $(arg gate_y) $(arg gate_z)"
+          opening_radius="$(arg gate_radius)" thickness="$(arg gate_thickness)"
+          material="mat_gate"/>
+    </xacro:if>
     <xacro:quadrotor_body prefix="$(arg quad_name)"
                           pos="$(arg init_x) $(arg init_y) $(arg init_z)"
