Commit message: Add configurable payload and gates to LiDAR simulation scene

File: model/scene_acro_payload_lidar.xml.xacro (robot description, xacro)
@@ -8,4 +8,27 @@
   <xacro:arg name="init_pitch" default="0.0"/>
   <xacro:arg name="init_yaw"   default="0.0"/>
+  <xacro:arg name="payload_x" default="-0.7"/>
+  <xacro:arg name="payload_y" default="0.0"/>
+  <xacro:arg name="payload_z" default="0.02"/>
+  <xacro:arg name="quadrotor_mass" default="1.24"/>
+  <xacro:arg name="quadrotor_ixx" default="0.0027338143976"/>
+  <xacro:arg name="quadrotor_iyy" default="0.0027336327812"/>
+  <xacro:arg name="quadrotor_izz" default="0.0052991944907"/>
+  <xacro:arg name="payload_mass" default="0.2"/>
+  <xacro:arg name="cable_length" default="0.95"/>
+  <!-- Optional gate: clear opening radius and full depth along world x. -->
+  <xacro:arg name="enable_gate" default="false"/>
+  <xacro:arg name="gate_x" default="2.0"/>
+  <xacro:arg name="gate_y" default="0.0"/>
+  <xacro:arg name="gate_z" default="2.0"/>
+  <xacro:arg name="gate_radius" default="0.4"/>
+  <xacro:arg name="gate_thickness" default="0.1"/>
+  <!-- Optional second gate for the multiple-gate TI-MPC planner. -->
+  <xacro:arg name="enable_second_gate" default="false"/>
+  <xacro:arg name="second_gate_x" default="3.5"/>
+  <xacro:arg name="second_gate_y" default="0.0"/>
+  <xacro:arg name="second_gate_z" default="2.0"/>
+  <xacro:arg name="second_gate_radius" default="0.4"/>
+  <xacro:arg name="second_gate_thickness" default="0.1"/>
   <xacro:arg name="meshdir" default="."/>
   <xacro:arg name="mesh_pos" default="-0.17 -0.16 -0.1"/>
@@ -28,4 +51,5 @@
   <xacro:arg name="acro_gyro_bias_rw" default="0.0"/>
   <xacro:include filename="quadrotor_acro_macro.xml.xacro" />
+  <xacro:include filename="circular_gate_macro.xml.xacro" />
   <compiler angle="radian" meshdir="$(arg meshdir)"/>
   <option timestep="$(arg simulation_timestep)" gravity="0 0 -9.81" density="1.225" viscosity="1.8e-05" integrator="RK4" />
@@ -57,4 +81,5 @@
     <material name="mat_cyan"   rgba="0.1 0.7 0.8 1" reflectance="0.01" shininess="0.01" specular="0.0" />
     <material name="mat_gray"   rgba="0.45 0.45 0.45 1" reflectance="0.01" shininess="0.01" specular="0.0" />
+    <material name="mat_gate" rgba="0.95 0.25 0.15 1" reflectance="0.05" shininess="0.05" specular="0.1"/>
     <xacro:quadrotor_visual_assets />
     <texture type="skybox" builtin="flat" rgb1="0 0 0" rgb2="0 0 0" width="512" height="3072"/>
@@ -72,4 +97,5 @@
     <geom class="environment" name="ceiling" type="box" pos="2.5 0 3.0" size="5.55 2.05 0.04" rgba="0.7 0.7 0.75 0.35"/>
     <geom class="environment" name="box_red" type="box" pos="2 1 0.1" size="0.2 0.2 0.1" material="mat_red" />
+    <geom class="environment" name="box_green" type="box" pos="4 -1 0.5" size="0.2 0.2 0.5" material="mat_green" />
     <geom class="environment" name="box_blue" type="box" pos="6 1 0.5" size="0.2 0.2 0.5" material="mat_blue" />
     <geom class="environment" name="pillar_cyan" type="cylinder" pos="1.2 -1.25 0.75" size="0.12 0.75" material="mat_cyan" />
@@ -79,16 +105,34 @@
     <geom class="environment" name="overhead_beam" type="box" pos="3.6 1.1 1.8" size="0.9 0.08 0.08" material="mat_gray" />
     <geom class="environment" name="offset_panel" type="box" pos="7.1 0.25 1.05" size="0.08 0.55 1.05" material="mat_red" />
+    <xacro:if value="$(arg enable_gate)">
+      <xacro:circular_gate name="planner_gate"
+          pos="$(arg gate_x) $(arg gate_y) $(arg gate_z)"
+          opening_radius="$(arg gate_radius)" thickness="$(arg gate_thickness)"
+          material="mat_gate"/>
+    </xacro:if>
+    <xacro:if value="$(arg enable_second_gate)">
+      <xacro:circular_gate name="planner_gate_2"
+          pos="$(arg second_gate_x) $(arg second_gate_y) $(arg second_gate_z)"
+          opening_radius="$(arg second_gate_radius)" thickness="$(arg second_gate_thickness)"
+          material="mat_gate"/>
+    </xacro:if>
+    <!-- Attach the cable 5 cm below the quadrotor body origin. -->
     <xacro:quadrotor_body prefix="$(arg quad_name)"
                           pos="$(arg init_x) $(arg init_y) $(arg init_z)"
                           euler="$(arg init_roll) $(arg init_pitch) $(arg init_yaw)"
+                          mass="$(arg quadrotor_mass)"
+                          ixx="$(arg quadrotor_ixx)"
+                          iyy="$(arg quadrotor_iyy)"
+                          izz="$(arg quadrotor_izz)"
                           mesh_pos="$(arg mesh_pos)"
                           mesh_euler="$(arg mesh_euler)"
                           primitive_alpha="$(arg primitive_alpha)"
+                          payload_site_pos="0.0 0.0 -0.05"
                           include_lidar="true" />
-    <body name="payload" pos="-0.7 0.0 0.02">
+    <body name="payload" pos="$(arg payload_x) $(arg payload_y) $(arg payload_z)">
       <joint name="payload_x" type="slide" axis="1 0 0" damping="0.06"/>
       <joint name="payload_y" type="slide" axis="0 1 0" damping="0.06"/>
       <joint name="payload_z" type="slide" axis="0 0 1" damping="0.06"/>
-      <geom type="sphere" size="0.035" rgba="0 0 1 0.8" mass="0.2"/>
+      <geom type="sphere" size="0.035" rgba="0 0 1 0.8" mass="$(arg payload_mass)"/>
       <site name="payload_connection_site" pos="0.0 0.0 0.0"/>
     </body>
@@ -109,5 +153,5 @@
   </actuator>
   <tendon>
-    <spatial name="rope0" limited="true" range="0 0.95" width=".0005">
+    <spatial name="rope0" limited="true" range="0 $(arg cable_length)" width=".0005">
       <site site="$(arg quad_name)_payload_site"/>
       <site site="payload_connection_site"/>
